File: uaefi.kicad_sch (KiCad schematic)
At the start: 44 parts, among them J1 USB_B_Mini, J1 USB_C_Receptacle_USB2.0, J1 rusefi_2x56_pin_conn, J5 Conn_01x05_Male, M1 Module-power_12and5V-0.2, M2 Module-vr-max9924-0.1, M3 Module-knock-0.2, M4 Module:mega-mcu100/0.2, M5 Module-lin-0.1, M6 Module-vr-max9924-0.1, M7 Module-vr-discrete-0.4, M9 Module-wbo-0.5

Commit message: Upd SCH
Parts:
- removed F6 (x3): 12H1500D, hellen-one-common:PAD-1206-PAD, symbol hellen-one-common:Fuse-Pad-Pad
- removed J1: rusefi_2x56_pin_conn, kicad6-libraries:rusefi_2x56_pin_connector, symbol rusefi_2x56_pin_connector:rusefi_2x56_pin_conn
- removed M2: Module-vr-max9924-0.1, hellen-one-vr-max9924-0.1:vr-max9924, symbol vr-max9924:Module-vr-max9924-0.1
- removed M3: Module-knock-0.2, hellen-one-knock-0.2:knock, symbol hellen-one-knock-0.2:Module-knock-0.2
- removed M5: Module-lin-0.1, hellen-one-lin-0.1:lin, symbol hellen-one-lin-0.1:Module-lin-0.1
- removed R1, R10, R11, R12, R13, R14, R15, R16, R2, R3, R4, R5, R54, R6, R7, R8, R9: Jumper-Pad-Pad, hellen-one-common:PAD-0805-PAD, symbol hellen-one-common:Jumper-Pad-Pad
- removed R30 (x2), R92: 4.7k, hellen-one-common:R0603, symbol hellen-one-common:Res
- added F6 (x4): 12H1500D, hellen-one-common:PAD-1206-PAD, symbol hellen-one-common:Fuse-Pad-Pad
- added H1, H2, H3, H4: M3, MountingHole:MountingHole_3.2mm_M3_Pad_Via, symbol Mechanical:MountingHole
- added J1, J7, J9: 5569-20A2, Connector_Molex:Molex_Mini-Fit_Jr_5569-20A2_2x10_P4.20mm_Horizontal, symbol Connector_Generic:Conn_02x10_Top_Bottom
- added J6, J8: 5569-06A2, Connector_Molex:Molex_Mini-Fit_Jr_5569-06A2_2x03_P4.20mm_Horizontal, symbol Connector_Generic:Conn_02x03_Top_Bottom
- added R30: 33k, hellen-one-common:R0603, symbol hellen-one-common:Res
- added R30: 6.8k, hellen-one-common:R0603, symbol hellen-one-common:Res
- added R30: 4.7k, hellen-one-common:R0603, symbol hellen-one-common:Res
- added R49, R50: Jumper-Pad-Pad, hellen-one-common:PAD-0805-PAD, symbol hellen-one-common:Jumper-Pad-Pad
- added R66: DNP, Resistor_SMD:R_2512_6332Metric, symbol hellen-one-common:Res
Connections:
- net IN_HALL4 is gone; now on net IN_BUTTON3: M4.S1 (IN_D4_(PE15))
- net +12V: now also F6.1, F6.1, F6.1, J8.4 (Pin_4), R30.2; no longer M1.E2 (V12)
- net +12V_RAW: now also F6.2, J6.3 (Pin_3)
- net +5VP: now also J1.1 (Pin_1), J1.2 (Pin_2), J9.1 (Pin_1), J9.2 (Pin_2), J9.5 (Pin_5), J9.6 (Pin_6), R30.1
- net CAN+: now also M4.W11 (CANH), J9.10 (Pin_10)
- net CAN-: now also M4.W12 (CANL), J9.9 (Pin_9)
- net DC Driver 1/DIR: now also M4.E21 (OUT_PWM4_(PC8))
- net DC Driver 1/PWM: now also M4.E20 (OUT_PWM3_(PC7))
- net DC Driver 1/PWR: now also F6.2
- net DC Driver 2/PWM: now also M4.E22 (OUT_PWM5_(PC9))
- net DC Driver 2/PWR: now also F6.2
- net GND: now also J7.1 (Pin_1), J7.11 (Pin_11), J8.1 (Pin_1)
- net GNDA: now also J1.11 (Pin_11), J1.12 (Pin_12), J9.11 (Pin_11), J9.12 (Pin_12), J9.15 (Pin_15), J9.16 (Pin_16), R30.1
- net IGN1: now also M4.W10 (IGN1_(PC13))
- net IGN2: now also M4.W9 (IGN2_(PE5))
- net IGN3: now also M4.W8 (IGN3_(PE4))
- net IGN4: now also M4.W7 (IGN4_(PE3))
- net INJ1: now also M4.E17 (OUT_INJ1_(PD3))
- net INJ2: now also M4.E16 (OUT_INJ2_(PA9))
- net INJ3: now also M4.E15 (OUT_INJ3_(PD11))
- net INJ4: now also M4.E14 (OUT_INJ4_(PD10))
- net IN_BUTTON1: now also M4.S14 (IN_CRANK_(PB1)), J1.4 (Pin_4)
- net IN_BUTTON2: now also M4.S16 (IN_CAM_(PA6)), J1.3 (Pin_3)
- net IN_BUTTON3: now also J1.13 (Pin_13)
- net IN_CLT: now also M4.S21 (IN_CLT_(PC2)), J9.7 (Pin_7)
- net IN_HALL1: now also J1.7 (Pin_7)
- net IN_HALL2: now also J1.6 (Pin_6)
- net IN_HALL3: now also J1.5 (Pin_5)
- net IN_IAT: now also M4.S20 (IN_IAT_(PC3)), J9.8 (Pin_8)
- net IN_KNOCK: now also J1.8 (Pin_8), R50.1; no longer M4.S15 (IN_KNOCK_(PA2))
- net IN_KNOCK_RAW: now also J1.14 (Pin_14)
- net IN_MAP: now also M4.S13 (IN_MAP1_(PC0)), J1.9 (Pin_9)
- net IN_PPS1: now also M4.S19 (IN_PPS_(PA3)), J9.4 (Pin_4)
- net IN_PPS2: now also M4.S8 (IN_AUX2_(PC4/PE9)), J9.3 (Pin_3)
- net IN_TLS115_PG: now also M4.E9 (SPI2_MOSI_(PB15))
- net IN_TPS1: now also M4.S18 (IN_TPS_(PA4)), J9.13 (Pin_13)
- net IN_TPS2: now also M4.S9 (IN_AUX1_(PB0)), J9.14 (Pin_14)
- net IN_VIGN: now also F6.2
- net OUT_IGN1: now also J7.7 (Pin_7)
- net OUT_IGN2: now also J7.6 (Pin_6)
- net OUT_IGN3: now also J7.5 (Pin_5)
- net OUT_IGN4: now also J7.4 (Pin_4)
- net OUT_INJ1: now also J7.17 (Pin_17)
- net OUT_INJ2: now also J7.16 (Pin_16)
- net OUT_INJ3: now also J7.15 (Pin_15)
- net OUT_INJ4: now also J7.14 (Pin_14)
- net VR1: now also M4.N18 (UART8_RX_(PE0)); no longer M4.S14 (IN_CRANK_(PB1))
- net VR1+: now also J1.19 (Pin_19)
- net VR1-: now also J1.18 (Pin_18)
- net VR2: now also M4.N19 (UART8_TX_(PE1))
- net VR2+: now also J1.17 (Pin_17)
- net VR2-: now also J1.16 (Pin_16), R66.1
- net WBO_Heater: now also J6.6 (Pin_6)
- net WBO_Ip: now also J6.4 (Pin_4)
- net WBO_Rtrim: now also J6.5 (Pin_5)
- net WBO_Un: now also J6.1 (Pin_1)
- net WBO_Vm: now also J6.2 (Pin_2)
- net LS2: now reaches M4.E10 (OUT_INJ8_(PD12))
- net LS1: now reaches M4.E11 (OUT_INJ7_(PD15))
- net INJ6: now reaches M4.E12 (OUT_INJ6_(PA8))
- net INJ5: now reaches M4.E13 (OUT_INJ5_(PD2))
- net LS3: now reaches M4.E18 (OUT_PWM1_(PD13))
- net LS4: now reaches M4.E19 (OUT_PWM2_(PC6))
- net VR1_THRESHOLD: now reaches M4.E23 (OUT_PWM6_(PD14))
- net VR1_THRESHOLD: now also M7.E1 (Thresh_IN)
- net DC2_DIS: now reaches M4.E6 (SPI2_CS_/_CAN2_RX_(PB12))
- net DC2_DIR: now reaches M4.E7 (SPI2_SCK_/_CAN2_TX_(PB13))
- net DC1_DIS: now reaches M4.E8 (SPI2_MISO_(PB14))
- net EGT/SPI_SCK: now reaches M4.N10 (SPI3_SCK_(PC10))
- net EGT/SPI_SO: now reaches M4.N11 (SPI3_MISO_(PC11))
- net EGT/SPI_CS: now reaches M4.N9 (SPI3_CS_(PA15))
- net IN_AUX2: now reaches M4.S10 (IN_O2S2_(PA1))
- net IN_AUX2: now also J9.18 (Pin_18)
- net IN_AUX1: now reaches M4.S11 (IN_O2S_/_CAN_WAKEUP_(PA0))
- net IN_AUX1: now also J9.19 (Pin_19)
- net INTERNAL_MAP: now reaches M4.S12 (IN_MAP2_(PC1))
- net IN_FLEX: now reaches M4.S17 (IN_VSS_(PE11))
- net IN_FLEX: now also J1.15 (Pin_15)
- net IN_VMAIN: now reaches M4.S6 (IN_AUX4_(PA7))
- net IN_VMAIN: now also R30.1, R30.2
- net IN_AUX3: now reaches M4.S7 (IN_AUX3_(PC5))
- net IN_AUX3: now also J9.17 (Pin_17)
- net LS_WEAK2: now reaches M4.W3 (IGN8_(PE6))
- net LS_WEAK1: now reaches M4.W4 (IGN7_(PB9))
- net IGN6: now reaches M4.W5 (IGN6_(PB8))
- net IGN5: now reaches M4.W6 (IGN5_(PE2))
- net VR1_A: now reaches M7.E2 (OUT_A)
- net VR1_A: now also R49.1
- new net: F6.1, J9.20 (Pin_20)
- new net: R30.2, R66.2
- new net ADC3: M4.S15 (IN_KNOCK_(PA2)), R49.2, R50.2
- new net EGT+: J1.10 (Pin_10)
- new net EGT-: J1.20 (Pin_20)
- new net OUT_DC1+: J8.6 (Pin_6)
- new net OUT_DC1-: J8.5 (Pin_5)
- new net OUT_DC2+: J8.3 (Pin_3)
- new net OUT_DC2-: J8.2 (Pin_2)
- new net OUT_IGN5: J7.3 (Pin_3)
- new net OUT_IGN6: J7.2 (Pin_2)
- new net OUT_INJ5: J7.13 (Pin_13)
- new net OUT_INJ6: J7.12 (Pin_12)
- new net OUT_LS1: J7.8 (Pin_8)
- new net OUT_LS2: J7.20 (Pin_20)
- new net OUT_LS3: J7.19 (Pin_19)
- new net OUT_LS4: J7.18 (Pin_18)
- new net OUT_LS_WEAK1: J7.10 (Pin_10)
- new net OUT_LS_WEAK2: J7.9 (Pin_9)
- no-connect marks 72 -> 34
Other:
- added sheet EGT (egt.kicad_sch)
- sheet MAP ports: added OUT; removed none
- note added: "Install a 0 Ohm R45 resistor for using VR2- as a hall sensor input."
- note added: "Move the resistor from position R143 to R145 to enable the CAN WAKEUP function. The AUX1 analog input will be unavailable."
- note added: "Move the resistor from position R50 to R49 to use ADC3 for receiving the analog signal VR1 instead of the knock signal."
- note added: "TODO: 10k PU"
- note removed: "TLE9201 motor driver"
- moved on the sheet: BT1, D10, J1, J5, M1, M3, M4, M6, M7, M9, R3, R6

Commit message: Upd SCH
Parts:
- added J17: Conn_01x06, Connector_PinHeader_2.54mm:PinHeader_1x06_P2.54mm_Vertical, symbol Connector_Generic:Conn_01x06
- renumbered G4 to G1, G3 to G2, G1 to G3, G2 to G4, J9 to J1, J1 to J2, J6 to J3, J8 to J4, J7 to J5, M7 to M3, M6 to M4, M9 to M5, M4 to M6, R49 to R5, R50 to R6
Connections:
- net GND: now also J2.8 (Pin_8), R30.1, J17.3 (Pin_3)
- net GNDA: no longer R30.1
- net IN_KNOCK: no longer J2.8 (Pin_8)
- net at M5.W5 (nReset): now also J17.5 (Pin_5)
- net at M5.W6 (SWDIO): now also J17.4 (Pin_4)
- net at M5.W7 (SWCLK): now also J17.2 (Pin_2)
- net at M5.W8 (V33_OUT): now also J17.1 (Pin_1)
- net DC Driver 1/DIR renamed DC1_DIR
- net DC Driver 1/PWM renamed DC1_PWM
- net DC Driver 2/PWM renamed DC2_PWM
- no-connect marks 34 -> 31
Other:
- note added: "Install a 0 Ohm R4 resistor for using VR2- as a hall sensor input"
- note added: "Move the resistor from position R6 to R5 to use ADC3 for receiving the analog signal VR1 instead of the knock signal"
- note added: "Pin 8 may be used for shielding VR signals"
- note removed: "Install a 0 Ohm R45 resistor for using VR2- as a hall sensor input."
- note removed: "Move the resistor from position R50 to R49 to use ADC3 for receiving the analog signal VR1 instead of the knock signal."
- note removed: "TODO: 10k PU"
- moved on the sheet: F6, H1, H2, H3, H4, J1, J2, J3, J4, J5, M5, R30

Commit message: #6, #7, #8, #9
Parts:
- added C3: 100n, hellen-one-common:C0603, symbol hellen-one-common:Cap
- added M7: Module-can-0.1, hellen-one-can-0.1:can, symbol hellen-one-can-0.1:Module-can-0.1
- added P1, P2, P3, P4: Pad, hellen-one-common:PAD-TH, symbol hellen-one-common:Pad
- added U4: JDY-33, alphax-2ch:JDY-33, symbol JDY-33:JDY-33
Connections:
- net +3.3VA: now also C3.2, M7.V2 (CAN_VIO), U4.12 (3V3)
- net +5VA: now also M7.V1 (V5)
- net DC2_DIR: now also M6.N12 (SPI3_MOSI_(PC12)); no longer M6.E7 (SPI2_SCK_/_CAN2_TX_(PB13))
- net DC2_DIS: now also M6.N4 (USBID_(PA10)); no longer M6.E6 (SPI2_CS_/_CAN2_RX_(PB12))
- net GND: now also C3.1, M7.E1 (GND), U4.13 (GND)
- net at M6.N13 (UART2_TX_(PD5)): now also U4.2 (RXD)
- net at M6.N14 (UART2_RX_(PD6)): now also U4.1 (TXD)
- net at M6.N14a (LED_GREEN): now also P4.1 (Pin_1)
- net at M6.N14b (LED_YELLOW): now also P3.1 (Pin_1)
- new net: M6.E6 (SPI2_CS_/_CAN2_RX_(PB12)), M7.V6 (CAN_RX)
- new net: M6.E7 (SPI2_SCK_/_CAN2_TX_(PB13)), M7.V5 (CAN_TX)
- new net: M7.S1 (CANL), P1.1 (Pin_1)
- new net: M7.S2 (CANH), P2.1 (Pin_1)
- no-connect marks 31 -> 27
Other:
- note added: "Bluetooth Module"
- note added: "MAX current 2A"
- note removed: "Maximum current 2A"

Commit message: Placement
Parts:
- removed R5, R6: Jumper-Pad-Pad, hellen-one-common:PAD-0805-PAD, symbol hellen-one-common:Jumper-Pad-Pad
- added P5, P6: Pad, hellen-one-common:PAD-TH, symbol hellen-one-common:Pad
- added R30 (x2): 0, hellen-one-common:R0603, symbol hellen-one-common:Res
- U4: footprint alphax-2ch:JDY-33 -> kicad6-libraries:JDY-33
Connections:
- net ADC3: now also R30.2, R30.2
- net GND: now also J5.10 (Pin_10), J5.20 (Pin_20); no longer J5.1 (Pin_1), J5.11 (Pin_11)
- net IN_KNOCK: now also R30.1
- net OUT_IGN1: now also J5.16 (Pin_16); no longer J5.7 (Pin_7)
- net OUT_IGN2: now also J5.15 (Pin_15); no longer J5.6 (Pin_6)
- net OUT_IGN3: now also J5.14 (Pin_14); no longer J5.5 (Pin_5)
- net OUT_IGN4: now also J5.13 (Pin_13); no longer J5.4 (Pin_4)
- net OUT_IGN5: now also J5.12 (Pin_12); no longer J5.3 (Pin_3)
- net OUT_IGN6: now also J5.11 (Pin_11); no longer J5.2 (Pin_2)
- net OUT_INJ1: now also J5.6 (Pin_6); no longer J5.17 (Pin_17)
- net OUT_INJ2: now also J5.5 (Pin_5); no longer J5.16 (Pin_16)
- net OUT_INJ3: now also J5.4 (Pin_4); no longer J5.15 (Pin_15)
- net OUT_INJ4: now also J5.3 (Pin_3); no longer J5.14 (Pin_14)
- net OUT_INJ5: now also J5.2 (Pin_2); no longer J5.13 (Pin_13)
- net OUT_INJ6: now also J5.1 (Pin_1); no longer J5.12 (Pin_12)
- net OUT_LS1: now also J5.7 (Pin_7); no longer J5.8 (Pin_8)
- net OUT_LS2: now also J5.19 (Pin_19); no longer J5.20 (Pin_20)
- net OUT_LS3: now also J5.18 (Pin_18); no longer J5.19 (Pin_19)
- net OUT_LS4: now also J5.17 (Pin_17); no longer J5.18 (Pin_18)
- net OUT_LS_WEAK1: now also J5.9 (Pin_9); no longer J5.10 (Pin_10)
- net OUT_LS_WEAK2: now also J5.8 (Pin_8); no longer J5.9 (Pin_9)
- net VR1_A: now also R30.1
- net IN_TLS115_PG: no longer names the net of M6.E9 (SPI2_MOSI_(PB15))
- net IN_TLS115_PG: now also P5.1 (Pin_1); no longer M1.E6 (PG_5VP)
- new net: M1.E6 (PG_5VP), P6.1 (Pin_1)
- no-connect marks 27 -> 30
Other:
- moved on the sheet: C3

Commit message: Upd SCH
Parts:
- removed J1, J5: 5569-20A2, Connector_Molex:Molex_Mini-Fit_Jr_5569-20A2_2x10_P4.20mm_Horizontal, symbol Connector_Generic:Conn_02x10_Top_Bottom
- removed J4: 5569-06A2, Connector_Molex:Molex_Mini-Fit_Jr_5569-06A2_2x03_P4.20mm_Horizontal, symbol Connector_Generic:Conn_02x03_Top_Bottom
- added J10: 5569-16A2, Connector_Molex:Molex_Mini-Fit_Jr_5569-16A2_2x08_P4.20mm_Horizontal, symbol Connector_Generic:Conn_02x08_Top_Bottom
- added J4: 5569-08A2, Connector_Molex:Molex_Mini-Fit_Jr_5569-08A2_2x04_P4.20mm_Horizontal, symbol Connector_Generic:Conn_02x04_Top_Bottom
- added J5: 5569-18A2, Connector_Molex:Molex_Mini-Fit_Jr_5569-18A2_2x09_P4.20mm_Horizontal, symbol Connector_Generic:Conn_02x09_Top_Bottom
- J1: LCSC C13453 -> (none); MyComment (none) -> DNP
Connections:
- net +12V: now also J4.6 (Pin_6)
- net +5VP: now also J10.3 (Pin_3), J10.4 (Pin_4)
- net CAN+: now also J10.8 (Pin_8)
- net CAN-: now also J10.7 (Pin_7)
- net GND: now also J4.1 (Pin_1), J4.2 (Pin_2)
- net GNDA: now also J10.11 (Pin_11), J10.12 (Pin_12), J10.16 (Pin_16)
- net IN_AUX1: now also J10.15 (Pin_15)
- net IN_AUX2: now also J10.14 (Pin_14)
- net IN_AUX3: now also J10.13 (Pin_13)
- net IN_CLT: now also J10.5 (Pin_5)
- net IN_IAT: now also J10.6 (Pin_6)
- net IN_PPS1: now also J10.2 (Pin_2)
- net IN_PPS2: now also J10.1 (Pin_1)
- net IN_TPS1: now also J10.9 (Pin_9)
- net IN_TPS2: now also J10.10 (Pin_10)
- net OUT_DC1+: now also J4.8 (Pin_8)
- net OUT_DC1-: now also J4.7 (Pin_7)
- net OUT_DC2+: now also J4.4 (Pin_4)
- net OUT_DC2-: now also J4.3 (Pin_3)
- net OUT_IGN1: now also J5.15 (Pin_15)
- net OUT_IGN2: now also J5.14 (Pin_14)
- net OUT_IGN3: now also J5.13 (Pin_13)
- net OUT_IGN4: now also J5.12 (Pin_12)
- net OUT_IGN5: now also J5.11 (Pin_11)
- net OUT_IGN6: now also J5.10 (Pin_10)
- net OUT_INJ1: now also J5.6 (Pin_6)
- net OUT_INJ2: now also J5.5 (Pin_5)
- net OUT_INJ3: now also J5.4 (Pin_4)
- net OUT_INJ4: now also J5.3 (Pin_3)
- net OUT_INJ5: now also J5.2 (Pin_2)
- net OUT_INJ6: now also J5.1 (Pin_1)
- net OUT_LS1: now also J5.7 (Pin_7)
- net OUT_LS2: now also J5.18 (Pin_18)
- net OUT_LS3: now also J5.17 (Pin_17)
- net OUT_LS4: now also J5.16 (Pin_16)
- net OUT_LS_WEAK1: now also J5.9 (Pin_9)
- net OUT_LS_WEAK2: now also J5.8 (Pin_8)
- net at F6.1: now also J4.5 (Pin_5)
Other:
- note added: "A"
- note added: "B"
- note added: "C"
- note added: "D"
- note added: "E"
- moved on the sheet: F6, R30

Commit message: Export
Parts:
- removed R66: DNP, Resistor_SMD:R_2512_6332Metric, symbol hellen-one-common:Res
- added P7, P8: Pad, hellen-one-common:PAD-TH, symbol hellen-one-common:Pad
- R30: LCSC C23162 -> (none); MyComment (none) -> DNP
Connections:
- net +12V: now also J4.8 (Pin_8); no longer J4.6 (Pin_6)
- net +12V_RAW: now also J3.1 (Pin_1); no longer J3.3 (Pin_3)
- net CAN+: now also J10.7 (Pin_7); no longer J10.8 (Pin_8)
- net CAN-: now also J10.8 (Pin_8); no longer J10.7 (Pin_7)
- net DC Driver 1/PWR: now also F6.2; no longer F6.2
- net DC Driver 2/PWR: now also F6.2; no longer F6.2
- net DC2_DIR: now also M6.E9 (SPI2_MOSI_(PB15)); no longer M6.N12 (SPI3_MOSI_(PC12))
- net GND: now also J4.3 (Pin_3), J4.4 (Pin_4); no longer J4.1 (Pin_1), J4.2 (Pin_2)
- net GNDA: now also J2.13 (Pin_13); no longer J10.16 (Pin_16)
- net IN_AUX1: now also J10.1 (Pin_1); no longer J10.15 (Pin_15)
- net IN_AUX2: now also J2.3 (Pin_3); no longer J10.14 (Pin_14)
- net IN_AUX3: now also J2.15 (Pin_15); no longer J10.13 (Pin_13)
- net IN_BUTTON1: now also J10.2 (Pin_2); no longer J2.4 (Pin_4)
- net IN_BUTTON2: now also J10.10 (Pin_10); no longer J2.3 (Pin_3)
- net IN_BUTTON3: now also J2.9 (Pin_9); no longer J2.13 (Pin_13)
- net IN_CLT: now also J10.16 (Pin_16); no longer J10.5 (Pin_5)
- net IN_FLEX: now also J10.5 (Pin_5); no longer J2.15 (Pin_15)
- net IN_HALL1: now also J2.5 (Pin_5); no longer J2.7 (Pin_7)
- net IN_HALL3: now also J2.7 (Pin_7); no longer J2.5 (Pin_5)
- net IN_IAT: now also J10.15 (Pin_15); no longer J10.6 (Pin_6)
- net IN_KNOCK_RAW: now also J10.14 (Pin_14); no longer J2.14 (Pin_14)
- net IN_MAP: now also J10.9 (Pin_9); no longer J2.9 (Pin_9)
- net IN_PPS1: now also J10.6 (Pin_6); no longer J10.2 (Pin_2)
- net IN_PPS2: now also J2.4 (Pin_4); no longer J10.1 (Pin_1)
- net IN_TPS1: now also J10.13 (Pin_13); no longer J10.9 (Pin_9)
- net IN_TPS2: now also J2.14 (Pin_14); no longer J10.10 (Pin_10)
- net OUT_DC1+: now also J4.5 (Pin_5); no longer J4.8 (Pin_8)
- net OUT_DC1-: now also J4.1 (Pin_1); no longer J4.7 (Pin_7)
- net OUT_DC2+: now also J4.6 (Pin_6); no longer J4.4 (Pin_4)
- net OUT_DC2-: now also J4.2 (Pin_2); no longer J4.3 (Pin_3)
- net OUT_IGN3: now also J5.12 (Pin_12); no longer J5.13 (Pin_13)
- net OUT_IGN4: now also J5.11 (Pin_11); no longer J5.12 (Pin_12)
- net OUT_IGN5: now also J5.13 (Pin_13); no longer J5.11 (Pin_11)
- net VR1+: now also J2.18 (Pin_18); no longer J2.19 (Pin_19)
- net VR1-: now also J2.19 (Pin_19); no longer J2.18 (Pin_18)
- net VR2+: now also J2.16 (Pin_16); no longer J2.17 (Pin_17)
- net VR2-: now also J2.17 (Pin_17), R30.2; no longer J2.16 (Pin_16)
- net WBO_Heater: now also J3.3 (Pin_3); no longer J3.6 (Pin_6)
- net WBO_Ip: now also J3.5 (Pin_5); no longer J3.4 (Pin_4)
- net WBO_Rtrim: now also J3.2 (Pin_2); no longer J3.5 (Pin_5)
- net WBO_Un: now also J3.4 (Pin_4); no longer J3.1 (Pin_1)
- net WBO_Vm: now also J3.6 (Pin_6); no longer J3.2 (Pin_2)
- net at F6.1: now also J4.7 (Pin_7); no longer J4.5 (Pin_5)
- net at P5.1 (Pin_1): now also M6.N12 (SPI3_MOSI_(PC12)); no longer M6.E9 (SPI2_MOSI_(PB15))
- net at M6.N13 (UART2_TX_(PD5)), U4.2 (RXD): now also P8.1 (Pin_1)
- net at M6.N14 (UART2_RX_(PD6)), U4.1 (TXD): now also P7.1 (Pin_1)
- net VREF1: now reaches M6.S22 (VREF1)
- net VREF1: now also M3.W2 (VREF)
- net VREF2: no longer names the net of M6.S5 (VREF2)
- net VREF2: no longer M3.W2 (VREF)
Other:
- note added: "Install a 4.7 kOhm R1 resistor for using VR2- as a hall sensor input"
- note removed: "Install a 0 Ohm R4 resistor for using VR2- as a hall sensor input"
- moved on the sheet: F6, P5, R30

Commit message: #16
Parts:
- J17: LCSC (none) -> C37208
Changed lines of the file:
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@@
+      (effects (font (size 1.27 1.27)) hide)
+    )
+    (property "LCSC" "C37208" (at 121.92 49.53 0)
       (effects (font (size 1.27 1.27)) hide)
     )
