File: uaefi.kicad_sch (KiCad schematic)
At the start: 47 parts, among them J1 USB_B_Mini, J1 USB_C_Receptacle_USB2.0, J10 5569-16A2, J17 Conn_01x06, J2 5569-20A2, J3 5569-06A2, J4 5569-08A2, J5 5569-18A2, J5 Conn_01x05_Male, M1 Module-power_12and5V-0.2, M3 Module-knock-0.2, M3 Module-vr-discrete-0.4, M4 Module-vr-max9924-0.1, M5 Module-wbo-0.5, M6 Module:mega-mcu100/0.2, M7 Module-can-0.1, P1 Pad, P2 Pad, P3 Pad, P4 Pad, P5 Pad, P6 Pad, P7 Pad, P8 Pad, U4 JDY-33

Commit message: #18 #19 #20
Parts:
- removed P5, P6: Pad, hellen-one-common:PAD-TH, symbol hellen-one-common:Pad
- added R4: Jumper-Pad-Pad, hellen-one-common:PAD-0805-PAD, symbol hellen-one-common:Jumper-Pad-Pad
Connections:
- net PG_5VP: now reaches M6.N12 (SPI3_MOSI_(PC12))
- net PG_5VP: now also R4.2
- net at M1.E6 (PG_5VP): now also R4.1
Changed lines of the file:
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@@
   (junction (at 255.27 138.43) (diameter 0) (color 0 0 0 0)
   )
-  (junction (at 27.94 182.88) (diameter 0) (color 0 0 0 0)
-  )
   (junction (at 67.31 238.76) (diameter 0) (color 0 0 0 0)
   )
@@
     (stroke (width 0.3048) (type solid) (color 0 194 194 1))
   )
+  (wire (pts (xy 256.54 116.84) (xy 248.92 116.84))
+    (stroke (width 0) (type default))
+  )
   (wire (pts (xy 63.5 218.44) (xy 77.47 218.44))
     (stroke (width 0) (type default))
@@
     (stroke (width 0) (type default))
   )
+  (wire (pts (xy 132.08 317.5) (xy 140.97 317.5))
+    (stroke (width 0) (type default))
+  )
   (bus (pts (xy 13.97 218.44) (xy 13.97 223.52))
     (stroke (width 0) (type default) (color 194 194 0 1))
@@
     (stroke (width 0) (type default))
   )
-  (wire (pts (xy 29.21 182.88) (xy 27.94 182.88))
-    (stroke (width 0) (type default))
-  )
   (wire (pts (xy 171.45 215.9) (xy 180.34 215.9))
     (stroke (width 0) (type default))
@@
     (effects (font (size 1.27 1.27)) (justify left bottom))
   )
+  (label "PG_5VP" (at 256.54 116.84 180) (fields_autoplaced)
+    (effects (font (size 1.27 1.27)) (justify right bottom))
+  )
   (label "IN_HALL1" (at 180.34 226.06 180) (fields_autoplaced)
     (effects (font (size 1.27 1.27)) (justify right bottom))
@@
     (effects (font (size 1.27 1.27)) (justify left bottom))
   )
-  (label "IN_BUTTON1" (at 29.21 182.88 180) (fields_autoplaced)
+  (label "IN_BUTTON1" (at 27.94 182.88 180) (fields_autoplaced)
     (effects (font (size 1.27 1.27)) (justify right bottom))
   )
@@
     (effects (font (size 1.27 1.27)) (justify left bottom))
   )
+  (label "PG_5VP" (at 140.97 317.5 180) (fields_autoplaced)
+    (effects (font (size 1.27 1.27)) (justify right bottom))
+  )
   (label "OUT_DC2+" (at 41.91 139.7 0) (fields_autoplaced)
     (effects (font (size 1.27 1.27)) (justify left bottom))
@@
     )
   )
+  (symbol (lib_id "hellen-one-common:Jumper-Pad-Pad") (at 127 317.5 0) (unit 1)
+    (in_bom yes) (on_board yes) (dnp no)
+    (property "Reference" "R4" (at 132.08 316.23 0)
+      (effects (font (size 1.016 1.016)))
+    )
+    (property "Value" "Jumper-Pad-Pad" (at 127 319.278 0)
+      (effects (font (size 1.016 1.016)) hide)
+    )
+    (property "Footprint" "hellen-one-common:PAD-0805-PAD" (at 127 321.31 0)
+      (effects (font (size 1.524 1.524)) hide)
+    )
+    (property "Datasheet" "" (at 127 317.5 0)
+      (effects (font (size 1.524 1.524)) hide)
+    )
+    (property "LCSC" "C17477" (at 127 321.31 0)
+      (effects (font (size 1.27 1.27)) hide)
+    )
+    (pin "1")
+    (pin "2")
+    (instances
+      (project "uaefi"
+        (path "/ac264c30-3e9a-4be2-b97a-9949b68bd497"
+          (reference "R4") (unit 1)
+        )
+      )
+    )
+  )
   (symbol (lib_id "Connector_Generic:Conn_02x08_Top_Bottom") (at 33.02 177.8 0) (mirror x) (unit 1)
     (in_bom yes) (on_board yes) (dnp no)
@@
     )
   )
-  (symbol (lib_id "hellen-one-common:Pad") (at 254 116.84 0) (unit 1)
-    (in_bom yes) (on_board yes) (dnp no)
-    (property "Reference" "P5" (at 255.27 116.84 0)
-      (effects (font (size 1.27 1.27)) (justify left))
-    )
-    (property "Value" "Pad" (at 254 119.38 0)
-      (effects (font (size 1.27 1.27)) hide)
-    )
-    (property "Footprint" "hellen-one-common:PAD-TH" (at 254 120.65 0)
-      (effects (font (size 1.27 1.27)) hide)
-    )
-    (property "Datasheet" "~" (at 254 116.84 0)
-      (effects (font (size 1.27 1.27)) hide)
-    )
-    (pin "1")
-    (instances
-      (project "uaefi"
-        (path "/ac264c30-3e9a-4be2-b97a-9949b68bd497"
-          (reference "P5") (unit 1)
-        )
-      )
-    )
-  )
   (symbol (lib_id "hellen-one-common:+12V_RAW") (at 99.06 134.62 0) (unit 1)
     (in_bom yes) (on_board yes) (dnp no)
@@
         )
       )
-    )
-  )
-  (symbol (lib_id "hellen-one-common:Pad") (at 127 317.5 0) (unit 1)
-    (in_bom yes) (on_board yes) (dnp no)
-    (property "Reference" "P6" (at 128.27 317.5 0)
-      (effects (font (size 1.27 1.27)) (justify left))
-    )
-    (property "Value" "Pad" (at 127 320.04 0)
-      (effects (font (size 1.27 1.27)) hide)
-    )
-    (property "Footprint" "hellen-one-common:PAD-TH" (at 127 321.31 0)
-      (effects (font (size 1.27 1.27)) hide)
-    )
-    (property "Datasheet" "~" (at 127 317.5 0)
-      (effects (font (size 1.27 1.27)) hide)
-    )
-    (pin "1")
-    (instances
-      (project "uaefi"
-        (path "/ac264c30-3e9a-4be2-b97a-9949b68bd497"
-          (reference "P6") (unit 1)
-        )
-      )

Commit message: upd
Parts:
- added P13, P14, P15, P16, P17, P18, P19, P20: Pad, hellen-one-common:PAD-TH, symbol hellen-one-common:Pad
Connections:
- net CAN+: now also P14.1 (Pin_1)
- net CAN-: now also P13.1 (Pin_1)
- net IN_CLT: now also P17.1 (Pin_1)
- net IN_FLEX: now also P16.1 (Pin_1)
- net IN_IAT: now also P18.1 (Pin_1)
- net IN_KNOCK_RAW: now also P19.1 (Pin_1)
- net IN_PPS1: now also P15.1 (Pin_1)
- net IN_TPS1: now also P20.1 (Pin_1)

Commit message: Upd PCB
Parts:
- added R38 (x3): 10k, hellen-one-common:R0805, symbol hellen-one-common:Res
- added R38, R39, R41: DNP, hellen-one-common:R0805, symbol hellen-one-common:Res
- M6: value Module:mega-mcu100/0.2 -> Module:mega-mcu100/0.3; footprint hellen-one-mega-mcu100-0.2:mega-mcu100 -> hellen-one-mega-mcu100-0.3:mega-mcu100; symbol hellen-one-mega-mcu100-0.2:Module{colon}mega-mcu100/0.2 -> hellen-one-mega-mcu100-0.3:Module{colon}mega-mcu100/0.3
Connections:
- net +5VA: now also R38.2, R38.2, R38.2
- net GNDA: now also R38.1, R39.1, R41.1
- net IN_BUTTON1: now also R38.1, R38.2
- net IN_BUTTON2: now also R38.1, R39.2
- net IN_BUTTON3: now also R38.1, R41.2
Other:
- note added: "Configurable "BUTTON" pulls"
- note added: "Pin Name Recommended function B8 OUT_LS_WEAK2 Fan Relay B9 OUT_LS_WEAK1 Main Relay B16 OUT_LS4 Fuel Pump Replay B18 OUT_LS2 Idle Air Valve C8 GND VR Shield C16 IN_AUX3 Fuel Pressure D10 IN_BUTTON2 A/C Request"
- title: hellen-112-17 -> UAEFI

Commit message: Upd PCB
Parts:
- removed P13, P14, P15, P16, P17, P18, P19, P20: Pad, hellen-one-common:PAD-TH, symbol hellen-one-common:Pad
- added J1, J11, J12, J13, J14, J15, J16, J17, J18, J19, J20, J21, J22, J24: Conn_02x02_Odd_Even, Connector_PinSocket_2.54mm:PinSocket_2x02_P2.54mm_Vertical, symbol Connector_Generic:Conn_02x02_Odd_Even
Connections:
- net +12V: now also J22.1 (Pin_1)
- net +12V_RAW: now also J24.1 (Pin_1)
- net +5VA: now also R38.2, R39.2, R41.2; no longer R38.2, R38.2, R38.2
- net +5VP: now also J12.1 (Pin_1), J12.2 (Pin_2), J14.1 (Pin_1), J14.2 (Pin_2)
- net CAN+: now also J1.2 (Pin_2)
- net CAN-: now also J1.1 (Pin_1)
- net GND: now also J17.1 (Pin_1), J22.2 (Pin_2), J22.4 (Pin_4)
- net GNDA: now also R38.1, R38.1, R38.1, J12.3 (Pin_3), J12.4 (Pin_4), J14.3 (Pin_3), J14.4 (Pin_4), J15.4 (Pin_4); no longer R38.1, R39.1, R41.1
- net IN_AUX1: now also J13.2 (Pin_2)
- net IN_AUX2: now also J15.2 (Pin_2)
- net IN_AUX3: now also J16.4 (Pin_4)
- net IN_BUTTON1: now also R38.1, R38.2, J13.1 (Pin_1); no longer R38.1, R38.2
- net IN_BUTTON2: now also R38.2, R39.1, J13.3 (Pin_3); no longer R38.1, R39.2
- net IN_BUTTON3: now also R38.2, R41.1; no longer R38.1, R41.2
- net IN_CLT: now also J1.3 (Pin_3)
- net IN_FLEX: now also J11.2 (Pin_2)
- net IN_HALL1: now also J16.2 (Pin_2)
- net IN_HALL2: now also J16.1 (Pin_1)
- net IN_HALL3: now also J17.2 (Pin_2)
- net IN_IAT: now also J1.4 (Pin_4)
- net IN_KNOCK_RAW: now also J11.3 (Pin_3)
- net IN_MAP: now also J13.4 (Pin_4)
- net IN_PPS1: now also J11.1 (Pin_1)
- net IN_PPS2: now also J15.1 (Pin_1)
- net IN_TPS1: now also J11.4 (Pin_4)
- net IN_TPS2: now also J15.3 (Pin_3)
- net OUT_IGN1: now also J19.3 (Pin_3)
- net OUT_IGN2: now also J20.1 (Pin_1)
- net OUT_IGN3: now also J21.1 (Pin_1)
- net OUT_IGN4: now also J21.3 (Pin_3)
- net OUT_IGN5: now also J20.3 (Pin_3)
- net OUT_INJ1: now also J19.4 (Pin_4)
- net OUT_INJ2: now also J20.2 (Pin_2)
- net OUT_INJ3: now also J20.4 (Pin_4)
- net OUT_INJ4: now also J21.2 (Pin_2)
- net OUT_INJ5: now also J21.4 (Pin_4)
- net OUT_LS1: now also J19.2 (Pin_2)
- net OUT_LS2: now also J18.1 (Pin_1)
- net OUT_LS3: now also J18.3 (Pin_3)
- net OUT_LS4: now also J19.1 (Pin_1)
- net OUT_LS_WEAK1: now also J18.2 (Pin_2)
- net OUT_LS_WEAK2: now also J18.4 (Pin_4)
- net VR1+: now also J17.3 (Pin_3)
- net VR2+: now also J16.3 (Pin_3)
- net VR2-: now also J17.4 (Pin_4)
- net WBO_Ip: now also J24.4 (Pin_4)
- net WBO_Rtrim: now also J24.3 (Pin_3)
- net WBO_Un: now also J24.2 (Pin_2)
- net 12V_KEY: now reaches F6.1, J4.7 (Pin_7)
- net 12V_KEY: now also J22.3 (Pin_3)
Other:
- moved on the sheet: R38, R39, R41

Commit message: Upd SCH, PCB
Parts:
- J1: value USB_C_Receptacle_USB2.0 -> USB_C; footprint Connector_USB:USB_C_Receptacle_XKB_U262-16XN-4BVC11 -> kicad6-libraries:USB_C; symbol Connector:USB_C_Receptacle_USB2.0 -> misc:USB_C
- U4: LCSC (none) -> C9900001612
Connections:
- net LS_WEAK1 renamed LS_HOT1
- net LS_WEAK2 renamed LS_HOT2
- net OUT_LS_WEAK1 renamed OUT_LS_HOT1
- net OUT_LS_WEAK2 renamed OUT_LS_HOT2
Other:
- sheet Low Side renamed LS HOT
- sheet Low Side 2A renamed LS
- sheet LS HOT: file LS_weak.kicad_sch -> LS_HOT.kicad_sch
- note added: "3.5A MAX Always hot capable"
- note added: "3.5A MAX Solenoid load capable"
- note added: "Pin Name Recommended function B8 OUT_LS_HOT2 Fan Relay B9 OUT_LS_HOT1 Main Relay B16 OUT_LS4 Fuel Pump Replay B18 OUT_LS2 Idle Air Valve C8 GND VR Shield C16 IN_AUX3 Fuel Pressure D10 IN_BUTTON2 A/C Request"
- note removed: "Low current Always hot capable"
- note removed: "MAX current 2A"
- note removed: "Pin Name Recommended function B8 OUT_LS_WEAK2 Fan Relay B9 OUT_LS_WEAK1 Main Relay B16 OUT_LS4 Fuel Pump Replay B18 OUT_LS2 Idle Air Valve C8 GND VR Shield C16 IN_AUX3 Fuel Pressure D10 IN_BUTTON2 A/C Request"
Changed lines of the file:
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@@
     (comment 1 "https://rusefi.com/s/uaefi")
   )
+  (junction (at 54.61 128.27) (diameter 0) (color 0 0 0 0)
+  )
   (junction (at 57.15 196.85) (diameter 0) (color 0 0 0 0)
   )
@@
   (junction (at 48.26 403.86) (diameter 0) (color 0 0 0 0)
   )
-  (junction (at 54.61 130.81) (diameter 0) (color 0 0 0 0)
-  )
   (junction (at 34.29 384.81) (diameter 0) (color 0 0 0 0)
   )
@@
     (stroke (width 0.3048) (type solid) (color 0 0 255 1))
   )
-  (bus (pts (xy 16.51 142.24) (xy 16.51 130.81))
+  (bus (pts (xy 16.51 142.24) (xy 16.51 128.27))
     (stroke (width 0) (type default) (color 0 194 194 1))
   )
@@
     (stroke (width 0) (type default) (color 255 153 0 1))
   )
-  (bus (pts (xy 54.61 130.81) (xy 109.22 130.81))
+  (bus (pts (xy 54.61 128.27) (xy 109.22 128.27))
     (stroke (width 0) (type default) (color 0 194 194 1))
   )
@@
     (stroke (width 0) (type default))
   )
-  (bus (pts (xy 54.61 130.81) (xy 54.61 142.24))
+  (bus (pts (xy 54.61 128.27) (xy 54.61 142.24))
     (stroke (width 0) (type default) (color 0 194 194 1))
   )
@@
     (stroke (width 0) (type default))
   )
-  (bus (pts (xy 16.51 130.81) (xy 54.61 130.81))
+  (bus (pts (xy 16.51 128.27) (xy 54.61 128.27))
     (stroke (width 0) (type default) (color 0 194 194 1))
   )
@@
     (stroke (width 0) (type default))
   )
-  (bus (pts (xy 109.22 130.81) (xy 109.22 161.29))
+  (bus (pts (xy 109.22 128.27) (xy 109.22 161.29))
     (stroke (width 0) (type default) (color 0 194 194 1))
   )
@@
     (effects (font (size 1.27 1.27)) (justify left bottom))
   )
+  (text "3.5A MAX\nSolenoid load\ncapable" (at 120.65 153.67 0)
+    (effects (font (size 1.27 1.27)) (justify left bottom))
+  )
   (text "D" (at 33.655 177.8 0)
     (effects (font (size 1.27 1.27)) (justify left bottom))
@@
     (effects (font (size 1.27 1.27)) (justify left bottom))
   )
-  (text "Pin	Name			Recommended function\nB8	OUT_LS_WEAK2	Fan Relay\nB9	OUT_LS_WEAK1	Main Relay\nB16	OUT_LS4			Fuel Pump Replay\nB18	OUT_LS2			Idle Air Valve\nC8  GND  			VR Shield\nC16	IN_AUX3			Fuel Pressure\nD10	IN_BUTTON2		A/C Request"
+  (text "Pin	Name			Recommended function\nB8	OUT_LS_HOT2		Fan Relay\nB9	OUT_LS_HOT1		Main Relay\nB16	OUT_LS4			Fuel Pump Replay\nB18	OUT_LS2			Idle Air Valve\nC8  GND  			VR Shield\nC16	IN_AUX3			Fuel Pressure\nD10	IN_BUTTON2		A/C Request"
     (at 63.5 109.22 0)
     (effects (font (size 1.27 1.27)) (justify left bottom))
@@
     (effects (font (size 1.27 1.27)) (justify right bottom))
   )
-  (text "Low current\nAlways hot\ncapable" (at 121.2103 112.8584 0)
+  (text "3.5A MAX\nAlways hot\ncapable" (at 121.2103 112.8584 0)
     (effects (font (size 1.27 1.27)) (justify left bottom))
   )
@@
     (effects (font (size 1.27 1.27)) (justify right bottom))
   )
-  (text "MAX current 2A" (at 120.3861 149.5824 0)
-    (effects (font (size 1.27 1.27)) (justify left bottom))
-  )
   (text "DC Motor" (at 259.08 36.83 0)
     (effects (font (size 1.27 1.27)) (justify right bottom))
@@
     (effects (font (size 1.27 1.27)) (justify left bottom))
   )
-  (label "OUT_LS_WEAK1" (at 26.67 355.6 180) (fields_autoplaced)
-    (effects (font (size 1.27 1.27)) (justify right bottom))
-  )
   (label "IN_BUTTON2" (at 34.29 341.63 0) (fields_autoplaced)
     (effects (font (size 1.27 1.27)) (justify left bottom))
@@
     (effects (font (size 1.27 1.27)) (justify left bottom))
   )
+  (label "OUT_LS_HOT1" (at 26.67 355.6 180) (fields_autoplaced)
+    (effects (font (size 1.27 1.27)) (justify right bottom))
+  )
   (label "VR1_THRESHOLD" (at 180.34 157.48 180) (fields_autoplaced)
     (effects (font (size 1.27 1.27)) (justify right bottom))
@@
     (effects (font (size 1.27 1.27)) (justify left bottom))
   )
-  (label "OUT_LS_WEAK1" (at 31.75 95.25 180) (fields_autoplaced)
+  (label "OUT_LS_HOT1" (at 31.75 95.25 180) (fields_autoplaced)
     (effects (font (size 1.27 1.27)) (justify right bottom))
   )
@@
     (effects (font (size 1.27 1.27)) (justify left bottom))
   )
-  (label "OUT_LS_WEAK2" (at 26.67 358.14 180) (fields_autoplaced)
+  (label "USB-" (at 241.3 325.12 180) (fields_autoplaced)
     (effects (font (size 1.27 1.27)) (justify right bottom))
   )
-  (label "USB-" (at 241.3 325.12 180) (fields_autoplaced)
+  (label "OUT_LS_HOT2" (at 31.75 97.79 180) (fields_autoplaced)
     (effects (font (size 1.27 1.27)) (justify right bottom))
   )
-  (label "OUT_LS_WEAK2" (at 31.75 97.79 180) (fields_autoplaced)
+  (label "OUT_LS_HOT2" (at 133.35 106.68 180) (fields_autoplaced)
     (effects (font (size 1.27 1.27)) (justify right bottom))
   )
@@
     (effects (font (size 1.27 1.27)) (justify left bottom))
   )
-  (label "OUT_LS_WEAK1" (at 120.65 104.14 0) (fields_autoplaced)
-    (effects (font (size 1.27 1.27)) (justify left bottom))
-  )
   (label "VBUS" (at 228.6 297.18 180) (fields_autoplaced)
     (effects (font (size 1.27 1.27)) (justify right bottom))
@@
     (effects (font (size 1.27 1.27)) (justify right bottom))
   )
+  (label "OUT_LS_HOT1" (at 133.35 104.14 180) (fields_autoplaced)
+    (effects (font (size 1.27 1.27)) (justify right bottom))
+  )
   (label "OUT_DC2+" (at 41.91 139.7 0) (fields_autoplaced)
     (effects (font (size 1.27 1.27)) (justify left bottom))
   )
-  (label "LS_WEAK2" (at 154.94 106.68 0) (fields_autoplaced)
+  (label "LS_HOT2" (at 154.94 106.68 0) (fields_autoplaced)
     (effects (font (size 1.27 1.27)) (justify left bottom))
   )
@@
     (effects (font (size 1.27 1.27)) (justify left bottom))
   )
-  (label "12V_MAIN" (at 33.02 363.22 0) (fields_autoplaced)
-    (effects (font (size 1.27 1.27)) (justify left bottom))
-  )
   (label "EGT+" (at 27.94 213.36 180) (fields_autoplaced)
     (effects (font (size 1.27 1.27)) (justify right bottom))
@@
     (effects (font (size 1.27 1.27)) (justify left bottom))
   )
-  (label "12V_MAIN" (at 41.91 134.62 0) (fields_autoplaced)
-    (effects (font (size 1.27 1.27)) (justify left bottom))
-  )
   (label "IN_HALL3" (at 27.94 220.98 180) (fields_autoplaced)
     (effects (font (size 1.27 1.27)) (justify right bottom))
@@
     (effects (font (size 1.27 1.27)) (justify left bottom))
   )
+  (label "OUT_LS_HOT2" (at 26.67 358.14 180) (fields_autoplaced)
+    (effects (font (size 1.27 1.27)) (justify right bottom))
+  )
   (label "VR1" (at 248.92 147.32 0) (fields_autoplaced)
     (effects (font (size 1.27 1.27)) (justify left bottom))
@@
     (effects (font (size 1.27 1.27)) (justify right bottom))
   )
-  (label "OUT_LS_WEAK2" (at 120.65 106.68 0) (fields_autoplaced)
-    (effects (font (size 1.27 1.27)) (justify left bottom))
-  )
   (label "CAN-" (at 255.27 129.54 180) (fields_autoplaced)
     (effects (font (size 1.27 1.27)) (justify right bottom))
@@
     (effects (font (size 1.27 1.27)) (justify right bottom))
   )
-  (label "LS_WEAK1" (at 154.94 104.14 0) (fields_autoplaced)
+  (label "LS_HOT1" (at 154.94 104.14 0) (fields_autoplaced)
     (effects (font (size 1.27 1.27)) (justify left bottom))
   )
@@
     )
   )
-  (symbol (lib_id "Connector:USB_C_Receptacle_USB2.0") (at 257.81 327.66 0) (mirror y) (unit 1)
+  (symbol (lib_id "misc:USB_C") (at 257.81 327.66 0) (mirror y) (unit 1)
     (in_bom yes) (on_board yes) (dnp no)
-    (property "Reference" "J1" (at 266.7 308.61 0)
+    (property "Reference" "J1" (at 248.92 308.61 0)
       (effects (font (size 1.27 1.27)))
     )
-    (property "Value" "USB_C_Receptacle_USB2.0" (at 257.81 308.61 0)
-      (effects (font (size 1.27 1.27)) hide)
+    (property "Value" "USB_C" (at 247.65 346.71 0)
+      (effects (font (size 1.27 1.27)) (justify right))
     )
-    (property "Footprint" "Connector_USB:USB_C_Receptacle_XKB_U262-16XN-4BVC11" (at 254 327.66 0)
+    (property "Footprint" "kicad6-libraries:USB_C" (at 254 327.66 0)
       (effects (font (size 1.27 1.27)) hide)
     )
@@
     )
   )
+  (symbol (lib_id "power:+12V") (at 33.02 363.22 270) (unit 1)
+    (in_bom yes) (on_board yes) (dnp no)
+    (property "Reference" "#PWR0111" (at 29.21 363.22 0)
+      (effects (font (size 1.27 1.27)) hide)
+    )
+    (property "Value" "+12V" (at 38.1 363.22 90)
+      (effects (font (size 1.27 1.27)))
+    )
+    (property "Footprint" "" (at 33.02 363.22 0)
+      (effects (font (size 1.27 1.27)) hide)
+    )
+    (property "Datasheet" "" (at 33.02 363.22 0)
+      (effects (font (size 1.27 1.27)) hide)
+    )
+    (pin "1")
+    (instances
+      (project "uaefi"
+        (path "/ac264c30-3e9a-4be2-b97a-9949b68bd497"
+          (reference "#PWR0111") (unit 1)
+        )
+      )
+    )
+  )
   (symbol (lib_id "Connector_Generic:Conn_02x08_Top_Bottom") (at 33.02 177.8 0) (mirror x) (unit 1)
     (in_bom yes) (on_board yes) (dnp no)
@@
       (effects (font (size 1.27 1.27)) (justify left bottom) hide)
     )
-    (property "LCSC" "" (at 266.7 154.94 0)
+    (property "LCSC" "C9900001612" (at 266.7 154.94 0)
       (effects (font (size 1.27 1.27)) hide)
     )
@@
       (effects (font (size 1.27 1.27)) hide)
     )
-    (property "Value" "+12V_RAW" (at 94.3483 130.1749 0)
+    (property "Value" "+12V_RAW" (at 93.98 130.81 0)
       (effects (font (size 1.27 1.27)) (justify left))
     )
@@
     (stroke (width 0.1524) (type solid))
     (fill (color 0 0 0 0.0000))
-    (property "Sheetname" "Low Side 2A" (at 146.05 149.86 90)
+    (property "Sheetname" "LS" (at 146.05 144.78 90)
       (effects (font (size 1.27 1.27)) (justify left bottom))
     )
@@
     (stroke (width 0.1524) (type solid))
     (fill (color 0 0 0 0.0000))
-    (property "Sheetname" "Low Side" (at 146.05 109.855 90)
+    (property "Sheetname" "LS HOT" (at 146.05 108.585 90)
       (effects (font (size 1.27 1.27)) (justify left bottom))
     )
-    (property "Sheetfile" "LS_weak.kicad_sch" (at 135.89 108.5346 0)
+    (property "Sheetfile" "LS_HOT.kicad_sch" (at 135.89 108.5346 0)
       (effects (font (size 1.27 1.27)) (justify left top) hide)
     )
