File: uaefi.kicad_sch (KiCad schematic)
At the start: 66 parts, among them J1 Conn_02x02_Odd_Even, J1 USB_B_Mini, J1 USB_C, J10 5569-16A2, J11 Conn_02x02_Odd_Even, J12 Conn_02x02_Odd_Even, J13 Conn_02x02_Odd_Even, J14 Conn_02x02_Odd_Even, J15 Conn_02x02_Odd_Even, J16 Conn_02x02_Odd_Even, J17 Conn_01x06, J17 Conn_02x02_Odd_Even, J18 Conn_02x02_Odd_Even, J19 Conn_02x02_Odd_Even, J2 5569-20A2, J20 Conn_02x02_Odd_Even, J21 Conn_02x02_Odd_Even, J22 Conn_02x02_Odd_Even, J24 Conn_02x02_Odd_Even, J3 5569-06A2, J4 5569-08A2, J5 5569-18A2, J5 Conn_01x05_Male, M1 Module-power_12and5V-0.2, M3 Module-knock-0.2, M3 Module-vr-discrete-0.4, M4 Module-vr-max9924-0.1, M5 Module-wbo-0.5, M6 Module:mega-mcu100/0.3, M7 Module-can-0.1, P1 Pad, P2 Pad, P3 Pad, P4 Pad, P7 Pad, P8 Pad, U4 JDY-33

Commit message: Rev C
Parts:
- removed M3: Module-vr-discrete-0.4, hellen-one-vr-discrete-0.4:vr-discrete, symbol hellen-one-vr-discrete-0.4:Module-vr-discrete-0.4
- added M3: Module-vr-discrete-0.5, hellen-one-vr-discrete-0.5:vr-discrete, symbol hellen-one-vr-discrete-0.5:Module-vr-discrete-0.5
Connections:
- net +5VA: now also M3.E4 (V5_IN)
- net GND: now also M3.G (GND)
- net VR1 renamed VR_DISCRETE
- net VR_DISCRETE: now also M3.E3 (OUT)
- net VR1+ renamed VR_DISCRETE+
- net VR_DISCRETE+: now also M3.W2 (VR+)
- net VR1- renamed VR_DISCRETE-
- net VR_DISCRETE-: now also M3.W1 (VR-)
- net VR1_A renamed VR_DISCRETE_A
- net VR_DISCRETE_A: now also M3.E2 (OUT_A)
- net VR1_THRESHOLD renamed VR_DISCRETE_THR
- net VR_DISCRETE_THR: now also M3.E1 (Thresh_IN)
- net VR2 renamed VR_MAX9924
- net VR2+ renamed VR_MAX9924+
- net VR2- renamed VR_MAX9924-
Other:
- note added: "Move the resistor from position R6 to R5 to use ADC3 for receiving the analog signal VR-DISCRETE instead of the knock signal"
- note removed: "Move the resistor from position R6 to R5 to use ADC3 for receiving the analog signal VR1 instead of the knock signal"
- moved on the sheet: C3, J17, R30

Commit message: #66
Parts:
- added P5, P6: Pad, hellen-one-common:PAD-TH, symbol hellen-one-common:Pad
Connections:
- net VR_DISCRETE: now also P5.1 (Pin_1)
- net VR_MAX9924: now also P6.1 (Pin_1)

Commit message: #62 #65 #66 #67 #53
Other:
- note added: "Pin Name Recommended function B8 OUT_LS_HOT2 Fan Relay B9 OUT_LS_HOT1 Main Relay B16 OUT_LS4 Fuel Pump Replay B18 OUT_LS2 Idle Air Valve C8 GND VR Shield C16 IN_AUX3 Fuel Pressure D10 IN_BUTTON2 A/C Request All inputs are 12V-tolerant"
- note removed: "Pin Name Recommended function B8 OUT_LS_HOT2 Fan Relay B9 OUT_LS_HOT1 Main Relay B16 OUT_LS4 Fuel Pump Replay B18 OUT_LS2 Idle Air Valve C8 GND VR Shield C16 IN_AUX3 Fuel Pressure D10 IN_BUTTON2 A/C Request"
Changed lines of the file:
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@@
 	(title_block
 		(title "UAEFI")
-		(date "2024-08-14")
+		(date "2024-08-15")
 		(rev "D")
 		(company "rusEFI.com")
@@
 		)
 	)
-	(text "Pin	Name			Recommended function\nB8	OUT_LS_HOT2		Fan Relay\nB9	OUT_LS_HOT1		Main Relay\nB16	OUT_LS4			Fuel Pump Replay\nB18	OUT_LS2			Idle Air Valve\nC8  GND  			VR Shield\nC16	IN_AUX3			Fuel Pressure\nD10	IN_BUTTON2		A/C Request"
+	(text "Pin	Name			Recommended function\nB8	OUT_LS_HOT2		Fan Relay\nB9	OUT_LS_HOT1		Main Relay\nB16	OUT_LS4			Fuel Pump Replay\nB18	OUT_LS2			Idle Air Valve\nC8  GND  			VR Shield\nC16	IN_AUX3			Fuel Pressure\nD10	IN_BUTTON2		A/C Request\n\nAll inputs are 12V-tolerant"
 		(exclude_from_sim no)
-		(at 63.5 109.22 0)
+		(at 62.484 86.36 0)
 		(effects
 			(font
 				(size 1.27 1.27)
 			)
-			(justify left bottom)
+			(justify left top)
 		)
 	)

Commit message: Rev E
Parts:
- removed M1: Module-power_12and5V-0.2, hellen-one-power_12and5V-0.2:power_12and5V, symbol hellen-one-power_12and5V:Module-power_12and5V-0.2
- added M1: Module-power_12and5V-0.3, hellen-one-power_12and5V-0.3:power_12and5V, symbol hellen-one-power_12and5V:Module-power_12and5V-0.3
Connections:
- net +12V_RAW: now also M1.V1 (V12_PERM), M1.V3 (V12_RAW)
- net +5V: now also M1.E4 (V5)
- net +5VP: now also M1.V4 (5VP)
- net GND: now also M1.S1 (GND)
- net IN_VIGN: now also M1.V2 (IN_VIGN)
- net PWR_EN: now also M1.E5 (EN_5VP)
- net VBAT: now also M1.E1 (VBAT)
- net VIGN: now also M1.E3 (VIGN)
- net at R4.1: now also M1.E6 (PG_5VP)
- net EGT/SPI_SCK renamed SCK3
- net EGT/SPI_SO renamed MISO3
Other:
- moved on the sheet: F6

Commit message: #81 #82 #86 #87
Parts:
- added D2, D3, D4, D5: B5819W, hellen-one-common:SOD-123, symbol hellen-one-common:1N4148WS
Connections:
- net +12V_RAW: now also D2.1 (K), D3.1 (K), D4.1 (K), D5.1 (K)
- net OUT_LS1: now also D2.2 (A)
- net OUT_LS2: now also D3.2 (A)
- net OUT_LS3: now also D4.2 (A)
- net OUT_LS4: now also D5.2 (A)
Other:
- note added: "Flyback diodes"
- note added: "Pin Name Recommended function B8 OUT_LS_HOT2 Fan Relay B9 OUT_LS_HOT1 Main Relay B16 OUT_LS4 Fuel Pump Replay B18 OUT_LS2 Idle Air Valve C8 GND VR Shield C15 IN_AUX3 Fuel Pressure D10 IN_BUTTON2 A/C Request All inputs are 12V-tolerant"
- note removed: "Pin Name Recommended function B8 OUT_LS_HOT2 Fan Relay B9 OUT_LS_HOT1 Main Relay B16 OUT_LS4 Fuel Pump Replay B18 OUT_LS2 Idle Air Valve C8 GND VR Shield C16 IN_AUX3 Fuel Pressure D10 IN_BUTTON2 A/C Request All inputs are 12V-tolerant"
- moved on the sheet: F6, R30

Commit message: #102
Connections:
- net WBO_Ip: no longer J3.5 (Pin_5), M5.E3 (LSU_Ip)
- net WBO_Rtrim: no longer J3.2 (Pin_2), M5.E4 (LSU_Rtrim)
- net WBO_Un: no longer J3.4 (Pin_4), M5.E1 (LSU_Un)
- net WBO_Heater renamed 3_WBO_Heater
- net WBO_Vm renamed 2_WBO_Vm
- new net 1_WBO_Ip: J3.5 (Pin_5), M5.E3 (LSU_Ip)
- new net 5_WBO_Rtrim: J3.2 (Pin_2), M5.E4 (LSU_Rtrim)
- new net 6_WBO_Un: J3.4 (Pin_4), M5.E1 (LSU_Un)
Other:
- note added: "4"
Changed lines of the file:
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@@
 	)
 	(bus_entry
-		(at 20.32 64.77)
+		(at 17.78 64.77)
 		(size -2.54 2.54)
 		(stroke
@@
 	)
 	(bus_entry
-		(at 20.32 62.23)
+		(at 17.78 62.23)
 		(size -2.54 2.54)
 		(stroke
@@
 	(wire
 		(pts
-			(xy 29.21 64.77) (xy 20.32 64.77)
+			(xy 29.21 64.77) (xy 17.78 64.77)
 		)
 		(stroke
@@
 	(bus
 		(pts
-			(xy 38.1 55.88) (xy 17.78 55.88)
+			(xy 38.1 55.88) (xy 15.24 55.88)
 		)
 		(stroke
@@
 		)
 	)
+	(bus
+		(pts
+			(xy 15.24 64.77) (xy 15.24 67.31)
+		)
+		(stroke
+			(width 0)
+			(type default)
+		)
+	)
 	(wire
 		(pts
@@
 	(bus
 		(pts
-			(xy 17.78 55.88) (xy 17.78 64.77)
+			(xy 15.24 55.88) (xy 15.24 64.77)
 		)
 		(stroke
@@
 	(wire
 		(pts
-			(xy 29.21 62.23) (xy 20.32 62.23)
+			(xy 29.21 62.23) (xy 17.78 62.23)
 		)
 		(stroke
@@
 		)
 	)
-	(bus
-		(pts
-			(xy 17.78 64.77) (xy 17.78 67.31)
-		)
-		(stroke
-			(width 0)
-			(type default)
-		)
-	)
 	(wire
 		(pts
@@
 		)
 	)
+	(text "4"
+		(exclude_from_sim no)
+		(at 25.146 67.31 0)
+		(effects
+			(font
+				(size 1.27 1.27)
+			)
+			(justify left bottom)
+		)
+	)
 	(text "Bluetooth Module"
 		(exclude_from_sim no)
@@
 		)
 	)
-	(label "WBO_Heater"
-		(at 40.64 39.37 0)
-		(effects
-			(font
-				(size 1.27 1.27)
-			)
-			(justify left bottom)
-		)
-	)
 	(label "IN_PPS1"
 		(at 95.25 339.09 0)
@@
 		)
 	)
+	(label "1_WBO_Ip"
+		(at 40.64 44.45 0)
+		(effects
+			(font
+				(size 1.27 1.27)
+			)
+			(justify left bottom)
+		)
+	)
 	(label "12V_KEY"
 		(at 41.91 137.16 0)
@@
 		)
 	)
-	(label "INJ4"
-		(at 154.94 127 0)
+	(label "3_WBO_Heater"
+		(at 40.64 39.37 0)
 		(effects
 			(font
@@
 		)
 	)
-	(label "VR_DISCRETE+"
-		(at 40.64 218.44 0)
+	(label "INJ4"
+		(at 154.94 127 0)
 		(effects
 			(font
@@
 		)
 	)
-	(label "WBO_Ip"
-		(at 40.64 44.45 0)
+	(label "VR_DISCRETE+"
+		(at 40.64 218.44 0)
 		(effects
 			(font
@@
 		)
 	)
-	(label "WBO_Un"
+	(label "6_WBO_Un"
 		(at 41.91 67.31 0)
 		(effects
@@
 		)
 	)
-	(label "WBO_Vm"
+	(label "2_WBO_Vm"
 		(at 41.91 62.23 0)
 		(effects
@@
 		)
 	)
-	(label "WBO_Ip"
+	(label "1_WBO_Ip"
 		(at 41.91 64.77 0)
 		(effects
@@
 		)
 	)
-	(label "WBO_Vm"
-		(at 40.64 46.99 0)
-		(effects
-			(font
-				(size 1.27 1.27)
-			)
-			(justify left bottom)
-		)
-	)
 	(label "IN_VIGN"
 		(at 63.5 309.88 0)
@@
 		)
 	)
-	(label "WBO_Rtrim"
-		(at 40.64 41.91 0)
-		(effects
-			(font
-				(size 1.27 1.27)
-			)
-			(justify left bottom)
-		)
-	)
 	(label "OUT_IGN2"
 		(at 44.45 105.41 0)
@@
 		)
 	)
+	(label "2_WBO_Vm"
+		(at 40.64 46.99 0)
+		(effects
+			(font
+				(size 1.27 1.27)
+			)
+			(justify left bottom)
+		)
+	)
 	(label "OUT_INJ2"
 		(at 31.75 105.41 180)
@@
 		)
 	)
+	(label "5_WBO_Rtrim"
+		(at 40.64 41.91 0)
+		(effects
+			(font
+				(size 1.27 1.27)
+			)
+			(justify left bottom)
+		)
+	)
 	(label "IN_MAP"
 		(at 180.34 200.66 180)
@@
 		)
 	)
+	(label "6_WBO_Un"
+		(at 40.64 49.53 0)
+		(effects
+			(font
+				(size 1.27 1.27)
+			)
+			(justify left bottom)
+		)
+	)
 	(label "CAN-"
 		(at 255.27 129.54 180)
@@
 		)
 	)
-	(label "WBO_Heater"
+	(label "3_WBO_Heater"
 		(at 29.21 62.23 180)
 		(effects
@@
 		)
 	)
-	(label "WBO_Rtrim"
+	(label "5_WBO_Rtrim"
 		(at 29.21 64.77 180)
 		(effects
@@
 		)
 	)
-	(label "WBO_Un"
-		(at 40.64 49.53 0)
-		(effects
-			(font
-				(size 1.27 1.27)
-			)
-			(justify left bottom)
-		)
-	)

Commit message: #106 #107 rev e2
Parts:
- removed F6 (x4): 12H1500D, hellen-one-common:PAD-1206-PAD, symbol hellen-one-common:Fuse-Pad-Pad
- removed R4: Jumper-Pad-Pad, hellen-one-common:PAD-0805-PAD, symbol hellen-one-common:Jumper-Pad-Pad
- added F1, F2, F3, F4: Fuse, Fuse:Fuse_1206_3216Metric_Pad1.42x1.75mm_HandSolder, symbol Device:Fuse
- M5: value Module-wbo-0.5 -> Module-wbo-0.6; footprint hellen-one-wbo-0.5:wbo -> hellen-one-wbo-0.6:wbo; symbol hellen-one-wbo-0.5:Module-wbo-0.5 -> hellen-one-wbo-0.6:Module-wbo-0.6
Connections:
- net WBO_Ip is gone; now on net 1_WBO_Ip: J24.4 (Pin_4)
- net WBO_Rtrim is gone; now on net 5_WBO_Rtrim: J24.3 (Pin_3)
- net WBO_Un is gone; now on net 6_WBO_Un: J24.2 (Pin_2)
- net +12V: now also F2.1, F3.1, F4.1
- net +12V_RAW: now also F2.2
- net 12V_KEY: now also F1.2
- net DC Driver 1/PWR: now also F4.2
- net DC Driver 2/PWR: now also F3.2
- net GND: no longer M5.E6 (LSU_H-)
- net IN_VIGN: now also F1.1
- net PG_5VP: now also M1.E6 (PG_5VP)
