File: uaefi.kicad_pcb (KiCad board)
At the start: 2 copper layers, 125 parts, among them J1 5569-20A2, J2 5569-20A2, J3 5569-06A2, J4 5569-06A2, J5 5569-20A2, J6 Conn_01x06, J7 Conn_01x05_Male, J8 USB_B_Mini, J9 USB_C_Receptacle_USB2.0, M1 Module-power_12and5V-0.2, M2 Module-knock-0.2, M3 Module-vr-discrete-0.4, M4 Module-vr-max9924-0.1, M6 Module:mega-mcu100/0.2, Q1 ZXMS6005SGTA, Q10 ISL9V3040D3S, Q11 ISL9V3040D3S, Q12 ISL9V3040D3S, Q13 ZXMS6005SGTA, Q14 ZXMS6005SGTA, Q15 ZXMS6005SGTA, Q16 ZXMS6005SGTA, Q17 ZXMS6005SGTA, Q18 ZXMS6005SGTA, Q2 ZXMS6005SGTA, Q3 ZXMS6005SGTA, Q4 ZXMS6005SGTA, Q5 AO3400A, Q6 AO3400A, Q7 ISL9V3040D3S, Q8 ISL9V3040D3S, Q9 ISL9V3040D3S, U1 TLE9201SG, U2 TLE9201SG, U3 MPX4/MPXH6400_MAP, U4 MAX31855KASA

Commit message: Placement
Parts:
- added C33: 100n, hellen-one-common:C0603, B.Cu at (147.0, 126.0)
- added M5: Module-wbo-0.5, hellen-one-wbo-0.5:wbo, F.Cu at (149.4, 120.4)
- added M7: Module-can-0.1, hellen-one-can-0.1:can, F.Cu at (80.6, 105.3)
- added P1: Pad, hellen-one-common:PAD-TH, F.Cu at (84.0, 102.5)
- added P2: Pad, hellen-one-common:PAD-TH, F.Cu at (81.0, 102.5)
- added P3: Pad, hellen-one-common:PAD-TH, F.Cu at (112.5, 157.5)
- added P4: Pad, hellen-one-common:PAD-TH, F.Cu at (112.5, 152.5)
- added P5: Pad, hellen-one-common:PAD-TH, F.Cu at (93.5, 128.5)
- added P6: Pad, hellen-one-common:PAD-TH, F.Cu at (93.5, 155.5)
- added U5: JDY-33, kicad6-libraries:JDY-33, F.Cu at (142.7, 138.7)
- BT1, C1, C10, C14, C15, C16, C17, C18, C19, C2, C20, C21, C22, C23, C29, C3, C4, C5, C6, C7, C8, C9, D1, D2, D4, D6, D7, D8, Q1, Q13, Q14, Q15, Q18, Q3, Q5, Q6, R1, R10, R12, R15, R16, R17, R18, R19, R2, R20, R21, R22, R23, R24, R25, R26, R27, R28, R29, R3, R30, R31, R32, R33, R34, R7, R8: moved to B.Cu
- R5, R6: value Jumper-Pad-Pad -> 0; footprint hellen-one-common:PAD-0805-PAD -> hellen-one-common:R0603
- moved R29 256.9 mm to (52.5, 122.0), turned to 90 degrees
- moved R31 253.0 mm to (55.0, 122.0), turned to 90 degrees
- moved H2 249.8 mm to (53.5, 156.5)
- moved R34 248.4 mm to (57.5, 122.0), turned to 90 degrees
- moved D2 245.0 mm to (69.0, 89.5), turned to 90 degrees
- moved D5 242.8 mm to (69.0, 91.0), turned to 90 degrees
- moved D3 242.4 mm to (69.0, 83.5), turned to 90 degrees
- moved D4 241.3 mm to (69.0, 82.0), turned to 90 degrees
- moved R10 241.0 mm to (69.5, 93.0)
- moved R12 238.7 mm to (69.0, 85.5)
- moved Q13 238.5 mm to (53.5, 94.0), turned to 90 degrees
- moved R13 238.3 mm to (69.5, 87.5)
- moved R11 237.5 mm to (69.5, 80.0)
- moved Q15 236.3 mm to (53.5, 103.0), turned to 90 degrees
- moved Q18 232.3 mm to (53.5, 112.0), turned to 90 degrees
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Connections:
- J5 pad 1: GND -> /OUT_INJ6
- J5 pad 10: /OUT_LS_WEAK1 -> GND
- J5 pad 11: GND -> /OUT_IGN6
- J5 pad 12: /OUT_INJ6 -> /OUT_IGN5
- J5 pad 13: /OUT_INJ5 -> /OUT_IGN4
- J5 pad 14: /OUT_INJ4 -> /OUT_IGN3
- J5 pad 15: /OUT_INJ3 -> /OUT_IGN2
- J5 pad 16: /OUT_INJ2 -> /OUT_IGN1
- J5 pad 17: /OUT_INJ1 -> /OUT_LS4
- J5 pad 18: /OUT_LS4 -> /OUT_LS3
- J5 pad 19: /OUT_LS3 -> /OUT_LS2
- J5 pad 2: /OUT_IGN6 -> /OUT_INJ5
- J5 pad 20: /OUT_LS2 -> GND
- J5 pad 3: /OUT_IGN5 -> /OUT_INJ4
- J5 pad 4: /OUT_IGN4 -> /OUT_INJ3
- J5 pad 5: /OUT_IGN3 -> /OUT_INJ2
- J5 pad 6: /OUT_IGN2 -> /OUT_INJ1
- J5 pad 7: /OUT_IGN1 -> /OUT_LS1
- J5 pad 8: /OUT_LS1 -> /OUT_LS_WEAK2
- J5 pad 9: /OUT_LS_WEAK2 -> /OUT_LS_WEAK1
- M1 pad E6: /IN_TLS115_PG -> Net-(M1-PG_5VP)
- M6 pad E6: /DC2_DIS -> Net-(M6-SPI2_CS_/_CAN2_RX_(PB12))
- M6 pad E7: /DC2_DIR -> Net-(M6-SPI2_SCK_/_CAN2_TX_(PB13))
- M6 pad E9: /IN_TLS115_PG -> Net-(M6-SPI2_MOSI_(PB15))
- M6 pad N12: unconnected-(M6-SPI3_MOSI_(PC12)-PadN12) -> /DC2_DIR
- M6 pad N13: unconnected-(M6-UART2_TX_(PD5)-PadN13) -> Net-(M6-UART2_TX_(PD5))
- M6 pad N14: unconnected-(M6-UART2_RX_(PD6)-PadN14) -> Net-(M6-UART2_RX_(PD6))
- M6 pad N14a: unconnected-(M6-LED_GREEN-PadN14a) -> Net-(M6-LED_GREEN)
- M6 pad N14b: unconnected-(M6-LED_YELLOW-PadN14b) -> Net-(M6-LED_YELLOW)
- M6 pad N4: unconnected-(M6-USBID_(PA10)-PadN4) -> /DC2_DIS
Other:
- board outline added: 100 x 100 mm

Commit message: Upd SCH
Parts:
- removed J1: 5569-20A2, Connector_Molex:Molex_Mini-Fit_Jr_5569-20A2_2x10_P4.20mm_Horizontal
- added J10: 5569-16A2, Connector_Molex:Molex_Mini-Fit_Jr_5569-16A2_2x08_P4.20mm_Horizontal, F.Cu at (110.3, 69.3)
- J4: value 5569-06A2 -> 5569-08A2; footprint Connector_Molex:Molex_Mini-Fit_Jr_5569-06A2_2x03_P4.20mm_Horizontal -> Connector_Molex:Molex_Mini-Fit_Jr_5569-08A2_2x04_P4.20mm_Horizontal
- J5: value 5569-20A2 -> 5569-18A2; footprint Connector_Molex:Molex_Mini-Fit_Jr_5569-20A2_2x10_P4.20mm_Horizontal -> Connector_Molex:Molex_Mini-Fit_Jr_5569-18A2_2x09_P4.20mm_Horizontal
- moved H1 8.50 mm to (53.5, 63.5)
- moved H4 8.50 mm to (146.5, 63.5)
- moved Q5 8.37 mm to (55.5, 76.4), turned to -90 degrees
- moved R15 5.40 mm to (56.7, 72.8)
- moved R16 5.40 mm to (54.2, 72.8)
- moved R29 4.12 mm to (50.9, 118.2)
- moved R31 4.12 mm to (53.4, 118.2)
- moved R34 4.12 mm to (55.9, 118.2)
- moved J5 3.60 mm to (59.3, 114.8)
- moved D7 3.10 mm to (56.0, 84.4)
- moved Q13 3.10 mm to (53.5, 90.9)
- moved Q15 3.10 mm to (53.5, 99.9)
- moved Q18 3.10 mm to (53.5, 108.9)
- moved Q6 3.10 mm to (52.0, 84.4)
- moved D6 2.55 mm to (55.5, 80.5)
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Connections:
- F1 pad 1: Net-(J1-Pin_20) -> Net-(J4-Pin_5)
- J4 pad 2: /OUT_DC2- -> GND
- J4 pad 3: /OUT_DC2+ -> /OUT_DC2-
- J4 pad 4: +12V -> /OUT_DC2+
- J4 pad 5: /OUT_DC1- -> Net-(J4-Pin_5)
- J4 pad 6: /OUT_DC1+ -> +12V
- J5 pad 10: GND -> /OUT_IGN6
- J5 pad 11: /OUT_IGN6 -> /OUT_IGN5
- J5 pad 12: /OUT_IGN5 -> /OUT_IGN4
- J5 pad 13: /OUT_IGN4 -> /OUT_IGN3
- J5 pad 14: /OUT_IGN3 -> /OUT_IGN2
- J5 pad 15: /OUT_IGN2 -> /OUT_IGN1
- J5 pad 16: /OUT_IGN1 -> /OUT_LS4
- J5 pad 17: /OUT_LS4 -> /OUT_LS3
- J5 pad 18: /OUT_LS3 -> /OUT_LS2
Other:
- board text added: "A"
- board text added: "Always looking for C/C++/PHP/Java developers https://rusefi.com/s/mission"
- board text added: "B"
- board text added: "C"
- board text added: "D"
- board text added: "E"
- board text added: "G G + - V"
- board text added: "SWD: R D G C V"
- board text added: "UAEFI rev. A"
- board text added: "USB"
- board text added: "https://rusefi.com/s/uaefu"

Commit message: Export
Parts:
- removed R4: DNP, Resistor_SMD:R_2512_6332Metric
- added P7: Pad, hellen-one-common:PAD-TH, F.Cu at (133.2, 136.0)
- added P8: Pad, hellen-one-common:PAD-TH, F.Cu at (133.2, 140.7)
- C27, L1, L2, R5, R6, U4: moved to B.Cu
- C28, C30: value 10nF 50V -> 10n; footprint Capacitor_SMD:C_0402_1005Metric -> hellen-one-common:C0603; moved to B.Cu
- C29: footprint Capacitor_SMD:C_0402_1005Metric -> hellen-one-common:C0603
- C31, C32: footprint Capacitor_SMD:C_0402_1005Metric -> hellen-one-common:C0603; moved to B.Cu
- R1: moved to F.Cu
- moved F1 84.3 mm to (72.8, 143.0)
- moved P5 29.7 mm to (93.5, 158.1)
- moved R29 9.63 mm to (60.5, 119.0), turned to 0 degrees
- moved C32 8.52 mm to (111.4, 86.5), turned to 90 degrees
- moved C31 7.26 mm to (109.6, 86.5)
- moved R31 7.14 mm to (60.5, 117.4), turned to 0 degrees
- moved D8 6.92 mm to (105.5, 80.4)
- moved C28 6.63 mm to (103.8, 77.4), turned to 0 degrees
- moved L2 6.43 mm to (104.5, 75.0)
- moved L1 5.51 mm to (106.5, 75.0)
- moved C27 5.40 mm to (111.8, 94.9)
- moved C30 4.55 mm to (107.2, 77.4), turned to 180 degrees
- moved P2 3.90 mm to (84.9, 102.5)
- moved R1 3.16 mm to (84.9, 80.1), turned to 180 degrees
- moved R6 3.01 mm to (127.6, 89.2)
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Connections:
- C28 pad 1: Net-(U4-T-) -> GND
- C28 pad 2: GND -> Net-(U4-T-)
- C30 pad 1: Net-(U4-T+) -> GND
- C30 pad 2: GND -> Net-(U4-T+)
- C31 pad 1: +3.3VA -> GND
- C31 pad 2: GND -> +3.3VA
- C32 pad 1: +3.3VA -> GND
- C32 pad 2: GND -> +3.3VA
- D8 pad 1: Net-(U4-T+) -> Net-(U4-T-)
- D8 pad 2: Net-(U4-T-) -> Net-(U4-T+)
- F1 pad 1: Net-(J4-Pin_5) -> Net-(J4-Pin_7)
- F3 pad 2: /DC Driver 1/PWR -> /DC Driver 2/PWR
- F4 pad 2: /DC Driver 2/PWR -> /DC Driver 1/PWR
- J10 pad 1: /IN_PPS2 -> /IN_AUX1
- J10 pad 10: /IN_TPS2 -> /IN_BUTTON2
- J10 pad 13: /IN_AUX3 -> /IN_TPS1
- J10 pad 14: /IN_AUX2 -> /IN_KNOCK_RAW
- J10 pad 15: /IN_AUX1 -> /IN_IAT
- J10 pad 16: GNDA -> /IN_CLT
- J10 pad 2: /IN_PPS1 -> /IN_BUTTON1
- J10 pad 5: /IN_CLT -> /IN_FLEX
- J10 pad 6: /IN_IAT -> /IN_PPS1
- J10 pad 7: /CAN- -> /CAN+
- J10 pad 8: /CAN+ -> /CAN-
- J10 pad 9: /IN_TPS1 -> /IN_MAP
- J2 pad 13: /IN_BUTTON3 -> GNDA
- J2 pad 14: /IN_KNOCK_RAW -> /IN_TPS2
- J2 pad 15: /IN_FLEX -> /IN_AUX3
- J2 pad 16: /VR2- -> /VR2+
- J2 pad 17: /VR2+ -> /VR2-
- J2 pad 18: /VR1- -> /VR1+
- J2 pad 19: /VR1+ -> /VR1-
- J2 pad 3: /IN_BUTTON2 -> /IN_AUX2
- J2 pad 4: /IN_BUTTON1 -> /IN_PPS2
- J2 pad 5: /IN_HALL3 -> /IN_HALL1
- J2 pad 7: /IN_HALL1 -> /IN_HALL3
- J2 pad 9: /IN_MAP -> /IN_BUTTON3
- J3 pad 1: /WBO_Un -> +12V_RAW
- J3 pad 2: /WBO_Vm -> /WBO_Rtrim
- J3 pad 3: +12V_RAW -> /WBO_Heater
- J3 pad 4: /WBO_Ip -> /WBO_Un
- J3 pad 5: /WBO_Rtrim -> /WBO_Ip
- J3 pad 6: /WBO_Heater -> /WBO_Vm
- J4 pad 1: GND -> /OUT_DC1-
- J4 pad 2: GND -> /OUT_DC2-
- J4 pad 3: /OUT_DC2- -> GND
- J4 pad 4: /OUT_DC2+ -> GND
- J4 pad 5: Net-(J4-Pin_5) -> /OUT_DC1+
- J4 pad 6: +12V -> /OUT_DC2+
- J4 pad 7: /OUT_DC1- -> Net-(J4-Pin_7)
- J4 pad 8: /OUT_DC1+ -> +12V
- J5 pad 11: /OUT_IGN5 -> /OUT_IGN4
- J5 pad 12: /OUT_IGN4 -> /OUT_IGN3
- J5 pad 13: /OUT_IGN3 -> /OUT_IGN5
- M2 pad W2: /VREF2 -> /VREF1
- M6 pad E9: Net-(M6-SPI2_MOSI_(PB15)) -> /DC2_DIR
- M6 pad N12: /DC2_DIR -> Net-(M6-SPI3_MOSI_(PC12))
- M6 pad S22: unconnected-(M6-VREF1-PadS22) -> /VREF1
- M6 pad S5: /VREF2 -> unconnected-(M6-VREF2-PadS5)
- P5 pad 1: Net-(M6-SPI2_MOSI_(PB15)) -> Net-(M6-SPI3_MOSI_(PC12))
- R1 pad 2: Net-(R1-Pad2) -> /VR2-
Routing:
- net +12V_RAW: track 0.00 -> 245.6 mm, vias 0 -> 2
- net +5VP: track 0.00 -> 193.3 mm, vias 0 -> 2
- net +3.3VA: track 0.00 -> 169.4 mm, vias 0 -> 5
- net /LS_WEAK2: track 0.00 -> 146.8 mm, vias 0 -> 2
- net /LS_WEAK1: track 0.00 -> 140.1 mm, vias 0 -> 2
- net +5VA: track 0.00 -> 134.5 mm, vias 0 -> 5
- net GNDA: track 0.00 -> 119.5 mm, vias 0 -> 3
- net /EGT/SPI_CS: track 0.00 -> 111.5 mm, vias 0 -> 1
- net /EGT/SPI_SCK: track 0.00 -> 107.3 mm, vias 0 -> 1
- net +3.3V: track 0.00 -> 107.2 mm, vias 0 -> 8
- net /EGT/SPI_SO: track 0.00 -> 104.7 mm, vias 0 -> 1
- net /CAN+: track 0.00 -> 102.9 mm
- net /CAN-: track 0.00 -> 100.8 mm
- net /IN_TPS2: track 0.00 -> 88.1 mm
- net /IGN1: track 0.00 -> 85.6 mm, vias 0 -> 1
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- added copper zone on B.Cu, net /DC Driver 1/PWR
- added copper zone on B.Cu, net /DC Driver 2/PWR
- added copper zone on B.Cu, net GND
- added copper zone on F.Cu, net GND
- added copper zone on In1.Cu, net GND
- added copper zone on In2.Cu, net GND
Other:
- copper layers 2 -> 4
- board text added: "1"
- board text added: "10"
- board text added: "11"
- board text added: "12"
- board text added: "16"
- board text added: "18"
- board text added: "20"
- board text added: "3"
- board text added: "3.3"
- board text added: "4"
- board text added: "5"
- board text added: "6"
- board text added: "8"
- board text added: "9"
- board text added: "CAN2"
- board text added: "G"
- board text added: "H"
- board text added: "L"
- board text added: "UART2 RX TX"
- board text added: "Use plastic washers"
- board text added: "WBO"

Commit message: Upd PCB
Other:
- board text added: "+ EGT -"
- board text added: "12V"
- board text added: "5V"
- board text added: "AUX1"
- board text added: "AUX2"
- board text added: "AUX3"
- board text added: "BTN1"
- board text added: "BTN2"
- board text added: "BTN3"
- board text added: "CLT"
- board text added: "DC1+"
- board text added: "DC1-"
- board text added: "DC2+"
- board text added: "DC2-"
- board text added: "FLEX"
- board text added: "GND"
- board text added: "GNDA"
- board text added: "HALL1"
- board text added: "HALL2"
- board text added: "HALL3"
- board text added: "Heater"
- board text added: "IAT"
- board text added: "IGN1"
- board text added: "IGN2"
- board text added: "IGN3"
- board text added: "IGN4"
- board text added: "IGN5"
- board text added: "IGN6"
- board text added: "INJ1"
- board text added: "INJ2"
- board text added: "INJ3"
- board text added: "INJ4"
- board text added: "INJ5"
- board text added: "INJ6"
- board text added: "Ip"
- board text added: "KNOCK"
- board text added: "L CAN H"
- board text added: "LS1"
- board text added: "LS2"
- board text added: "LS3"
- board text added: "LS4"
- board text added: "LSW2"
- board text added: "LSW3"
- board text added: "MAP"
- board text added: "PPS1"
- board text added: "PPS2"
- board text added: "Rtrim"
- board text added: "TPS1"
- board text added: "TPS2"
- board text added: "Un"
- board text added: "VIGN"
- board text added: "VR1+"
- board text added: "VR1-"
- board text added: "VR2+"
- board text added: "VR2-"
- board text added: "Vm"

Commit message: #18 #19 #20
Parts:
- removed P5, P6: Pad, hellen-one-common:PAD-TH
- added R4: Jumper-Pad-Pad, hellen-one-common:PAD-0805-PAD, F.Cu at (93.5, 155.4)
Connections:
- M6 pad N12: Net-(M6-SPI3_MOSI_(PC12)) -> /PG_5VP
Routing:
- net /PG_5VP: track 0.00 -> 22.5 mm, vias 0 -> 2
- net Net-(M6-SPI3_MOSI_(PC12)): track 22.1 -> 0.00 mm, vias 2 -> 0
Other:
- outline, holes or cut-outs redrawn
