File: uaefi.kicad_pcb (KiCad board)
At the start: 4 copper layers, 100 x 100 mm, 135 parts, among them J10 5569-16A2, J2 5569-20A2, J3 5569-06A2, J4 5569-08A2, J5 5569-18A2, J6 Conn_01x06, J7 Conn_01x05_Male, J8 USB_B_Mini, J9 USB_C_Receptacle_USB2.0, M1 Module-power_12and5V-0.2, M2 Module-knock-0.2, M3 Module-vr-discrete-0.4, M4 Module-vr-max9924-0.1, M5 Module-wbo-0.5, M6 Module:mega-mcu100/0.2, M7 Module-can-0.1, P1 Pad, P2 Pad, P3 Pad, P4 Pad, P7 Pad, P8 Pad, Q1 ZXMS6005SGTA, Q10 ISL9V3040D3S, Q11 ISL9V3040D3S, Q12 ISL9V3040D3S, Q13 ZXMS6005SGTA, Q14 ZXMS6005SGTA, Q15 ZXMS6005SGTA, Q16 ZXMS6005SGTA, Q17 ZXMS6005SGTA, Q18 ZXMS6005SGTA, Q2 ZXMS6005SGTA, Q3 ZXMS6005SGTA, Q4 ZXMS6005SGTA, Q5 AO3400A, Q6 AO3400A, Q7 ISL9V3040D3S, Q8 ISL9V3040D3S, Q9 ISL9V3040D3S, U1 TLE9201SG, U2 TLE9201SG, U3 MPX4/MPXH6400_MAP, U4 MAX31855KASA, U5 JDY-33

Commit message: upd
Parts:
- added P10: Pad, hellen-one-common:PAD-TH, F.Cu at (128.0, 70.8)
- added P11: Pad, hellen-one-common:PAD-TH, F.Cu at (138.9, 73.4)
- added P12: Pad, hellen-one-common:PAD-TH, F.Cu at (136.4, 73.4)
- added P13: Pad, hellen-one-common:PAD-TH, F.Cu at (130.5, 73.3)
- added P14: Pad, hellen-one-common:PAD-TH, F.Cu at (128.0, 73.3)
- added P5: Pad, hellen-one-common:PAD-TH, F.Cu at (138.9, 70.8)
- added P6: Pad, hellen-one-common:PAD-TH, F.Cu at (136.4, 70.8)
- added P9: Pad, hellen-one-common:PAD-TH, F.Cu at (130.5, 70.8)
Routing:
- net /IN_PPS1: track 46.5 -> 47.4 mm
- net /CAN+: track 102.9 -> 103.4 mm
- net GND: vias 225 -> 223

Commit message: upd
Other:
- board text added: "COMMUNITY SUPPORT ECU"
- board text removed: "«COMMUNITY SUPPORT ECU»"
Changed lines of the file:
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@@
     (effects (font (size 1 1) (thickness 0.15)) (justify mirror))
   )
-  (gr_text "«COMMUNITY SUPPORT ECU»" (at 126.4 111) (layer "B.SilkS")
+  (gr_text "COMMUNITY SUPPORT ECU" (at 126.4 111) (layer "B.SilkS")
     (effects (font (size 1 1) (thickness 0.15)) (justify left bottom mirror))
   )
@@
     (effects (font (size 1 1) (thickness 0.15)))
   )
-  (gr_text "«COMMUNITY SUPPORT ECU»" (at 104.5 111.5) (layer "F.SilkS")
+  (gr_text "COMMUNITY SUPPORT ECU" (at 104.5 111.5) (layer "F.SilkS")
     (effects (font (size 1 1) (thickness 0.15)) (justify left bottom))
   )

Commit message: Upd PCB
Parts:
- added P15: Pad, hellen-one-common:PAD-TH, F.Cu at (55.5, 148.5)
- added P16: Pad, hellen-one-common:PAD-TH, F.Cu at (58.1, 148.5)
- added P17: Pad, hellen-one-common:PAD-TH, F.Cu at (53.0, 148.5)
- added P18: Pad, hellen-one-common:PAD-TH, F.Cu at (73.0, 149.0)
- added R35: 10k, hellen-one-common:R0805, F.Cu at (148.2, 69.5)
- added R36: 10k, hellen-one-common:R0805, F.Cu at (148.2, 72.0)
- added R37: 10k, hellen-one-common:R0805, F.Cu at (148.2, 74.5)
- added R38: DNP, hellen-one-common:R0805, F.Cu at (144.8, 69.5)
- added R39: DNP, hellen-one-common:R0805, F.Cu at (144.8, 72.0)
- added R40: DNP, hellen-one-common:R0805, F.Cu at (144.8, 74.5)
- M6: value Module:mega-mcu100/0.2 -> Module:mega-mcu100/0.3; footprint hellen-one-mega-mcu100-0.2:mega-mcu100 -> hellen-one-mega-mcu100-0.3:mega-mcu100
- Q10, Q11, Q12, Q7, Q8, Q9: value ISL9V3040D3S -> ISL9V3040D3ST
- moved C12 0.40 mm to (51.6, 145.8)
Connections:
- P10 pad 1: (no net) -> /IN_FLEX
- P11 pad 1: (no net) -> /IN_CLT
- P12 pad 1: (no net) -> /IN_IAT
- P13 pad 1: (no net) -> /IN_KNOCK_RAW
- P14 pad 1: (no net) -> /IN_TPS1
- P5 pad 1: (no net) -> /CAN-
- P6 pad 1: (no net) -> /CAN+
- P9 pad 1: (no net) -> /IN_PPS1
Routing:
- net /IN_BUTTON3: track 48.4 -> 109.6 mm, vias 0 -> 1
- net /IN_BUTTON1: track 46.0 -> 84.9 mm, vias 0 -> 1
- net +5VA: track 134.5 -> 171.1 mm, vias 5 -> 6
- net GNDA: track 119.5 -> 155.0 mm, vias 3 -> 5
- net /IN_BUTTON2: track 41.4 -> 76.4 mm, vias 0 -> 1
- net /DC1_PWM: track 38.2 -> 60.9 mm, vias 1 -> 2
- net /DC1_DIR: track 46.5 -> 64.0 mm
- net /DC2_DIR: track 52.8 -> 57.6 mm, vias 3 -> 2
- net /OUT_DC2-: track 35.7 -> 37.4 mm
- net /DC2_PWM: track 37.0 -> 38.3 mm, vias 1 -> 0
- net +5VP: track 193.3 -> 194.4 mm
- net /OUT_DC1-: track 20.4 -> 19.6 mm
- net /CAN+: track 103.4 -> 102.6 mm
- net +3.3V: track 107.2 -> 107.9 mm
- net GND: vias 223 -> 221
Other:
- board text added: "BT1"
- board text added: "BT2"
- board text added: "BT3"
- board text added: "DOWN"
- board text added: "UP"
