File: uaefi.kicad_pcb (KiCad board)
At the start: 4 copper layers, 100 x 100 mm, 158 parts, among them J1 Conn_02x02_Odd_Even, J10 5569-16A2, J11 Conn_02x02_Odd_Even, J12 Conn_02x02_Odd_Even, J13 Conn_02x02_Odd_Even, J14 Conn_02x02_Odd_Even, J15 Conn_02x02_Odd_Even, J16 Conn_02x02_Odd_Even, J17 Conn_02x02_Odd_Even, J18 Conn_02x02_Odd_Even, J19 Conn_02x02_Odd_Even, J2 5569-20A2, J20 Conn_02x02_Odd_Even, J21 Conn_02x02_Odd_Even, J22 Conn_02x02_Odd_Even, J24 Conn_02x02_Odd_Even, J3 5569-06A2, J4 5569-08A2, J5 5569-18A2, J6 Conn_01x06, J7 Conn_01x05_Male, J8 USB_B_Mini, J9 USB_C, M1 Module-power_12and5V-0.3, M2 Module-knock-0.2, M3 Module-vr-discrete-0.5, M4 Module-vr-max9924-0.1, M5 Module-wbo-0.6, M6 Module:mega-mcu100/0.3, M7 Module-can-0.1, P1 Pad, P15 Pad, P16 Pad, P17 Pad, P18 Pad, P2 Pad, P3 Pad, P4 Pad, P5 Pad, P6 Pad, P7 Pad, P8 Pad, Q10 ISL9V3040D3ST, Q11 ISL9V3040D3ST, Q12 ISL9V3040D3ST, Q7 ISL9V3040D3ST, Q8 ISL9V3040D3ST, Q9 ISL9V3040D3ST, U1 TLE9201SG, U10 VNLD5160TR-E, U11 VNLD5160TR-E, U2 TLE9201SG, U3 MPX4/MPXH6400_MAP, U4 MAX31855KASA, U5 JDY-33, U6 VNLD5160TR-E, U7 VNLD5160TR-E, U8 VNLD5160TR-E, U9 VNLD5160TR-E

Commit message: Unification with UAEFI F7 #114 #110
Parts:
- added R4: 4.7k, hellen-one-common:R0603, B.Cu at (53.6, 70.2)
- added R41: 4.7k, hellen-one-common:R0603, B.Cu at (56.5, 70.2)
- added R42: 4.7k, hellen-one-common:R0603, B.Cu at (51.3, 86.4)
- added R43: 4.7k, hellen-one-common:R0603, B.Cu at (53.8, 86.3)
- added R44: 4.7k, hellen-one-common:R0603, B.Cu at (52.5, 118.2)
- added R45: 4.7k, hellen-one-common:R0603, B.Cu at (86.2, 130.7)
- added R46: 4.7k, hellen-one-common:R0603, B.Cu at (62.0, 118.5)
- added R47: 4.7k, hellen-one-common:R0603, B.Cu at (55.9, 118.2)
- added R48: 4.7k, hellen-one-common:R0603, F.Cu at (78.6, 86.8)
- added R49: 4.7k, hellen-one-common:R0603, F.Cu at (80.2, 81.7)
- added R50: 4.7k, hellen-one-common:R0603, B.Cu at (79.5, 80.5)
- added R51: 4.7k, hellen-one-common:R0603, B.Cu at (80.3, 86.7)
- C25: moved to B.Cu
- moved C25 24.6 mm to (55.2, 130.0), turned to 0 degrees
- moved R13 3.10 mm to (80.3, 89.8)
- moved R11 2.39 mm to (81.0, 79.4), turned to 180 degrees
- moved R34 1.60 mm to (57.5, 118.2), turned to -90 degrees
- moved R31 1.55 mm to (51.0, 118.2), turned to -90 degrees
- moved M5 0.88 mm to (149.4, 120.1)
- moved R10 0.75 mm to (78.6, 88.3)
- moved R15 0.30 mm to (52.2, 70.1)
- turned F1 to -90 degrees
Connections:
- F1 pad 1: /IN_VIGN -> /12V_KEY
- F1 pad 2: /12V_KEY -> /IN_VIGN
- H1 pad 1: (no net) -> unconnected-(H1-Pad1)_4
- H2 pad 1: (no net) -> unconnected-(H2-Pad1)
- H3 pad 1: (no net) -> unconnected-(H3-Pad1)_6
- H4 pad 1: (no net) -> unconnected-(H4-Pad1)_7
- U10 pad 1: /INJ3 -> Net-(U10-IN1)
- U10 pad 3: /INJ4 -> Net-(U10-IN2)
- U11 pad 1: /INJ5 -> Net-(U11-IN1)
- U11 pad 3: /INJ6 -> Net-(U11-IN2)
- U4 pad 8: (no net) -> unconnected-(U4-NC-Pad8)
- U6 pad 1: /LS_HOT2 -> Net-(U6-IN1)
- U6 pad 3: /LS_HOT1 -> Net-(U6-IN2)
- U7 pad 1: /LS1 -> Net-(U7-IN1)
- U7 pad 3: /LS2 -> Net-(U7-IN2)
- U8 pad 1: /LS3 -> Net-(U8-IN1)
- U8 pad 3: /LS4 -> Net-(U8-IN2)
- U9 pad 1: /INJ1 -> Net-(U9-IN1)
- U9 pad 3: /INJ2 -> Net-(U9-IN2)
Routing:
- net Net-(U10-IN2): track 0.00 -> 70.4 mm, vias 0 -> 2
- net /INJ4: track 73.3 -> 12.7 mm, vias 2 -> 0
- net Net-(U11-IN1): track 0.00 -> 22.4 mm, vias 0 -> 2
- net /INJ3: track 79.3 -> 57.4 mm, vias 3 -> 2
- net Net-(U10-IN1): track 0.00 -> 21.4 mm, vias 0 -> 2
- net /INJ5: track 65.3 -> 46.2 mm
- net /INJ6: track 68.1 -> 56.3 mm, vias 3 -> 2
- net Net-(U11-IN2): track 0.00 -> 11.7 mm, vias 0 -> 2
- net /INJ1: track 88.9 -> 94.1 mm
- net /LS4: track 76.8 -> 72.1 mm
- net /LS_HOT1: track 140.6 -> 143.7 mm
- net /INJ2: track 81.7 -> 84.8 mm
- net Net-(U6-IN2): track 0.00 -> 2.89 mm
- net /LS_HOT2: track 138.9 -> 141.8 mm
- net Net-(U8-IN2): track 0.00 -> 2.86 mm
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Other:
- board text added: "UAEFI"
- board text added: "rev. f"
- board text removed: "UAEFI rev. E2"

Commit message: #118 #110 skip rev f
Parts:
- added G***: LOGO, LOGO, B.Cu at (122.8, 96.1)
- moved R6 2.42 mm to (125.4, 88.2), turned to 180 degrees
Routing:
- net /ADC3: track 43.7 -> 46.9 mm
- net /IN_KNOCK: track 1.56 -> 2.08 mm
Other:
- board text added: "rev. f2"
- board text removed: "rev. f"

Commit message: #120 moved
Parts:
- moved R16 4.97 mm to (58.0, 74.2)
- moved R15 3.30 mm to (55.5, 70.1), turned to 0 degrees
- moved R41 1.89 mm to (58.0, 71.3), turned to 90 degrees
- moved U5 1.68 mm to (142.2, 137.3)
- moved BT1 1.65 mm to (142.1, 132.8)
- moved D1 1.51 mm to (138.2, 142.5)
- moved M5 1.28 mm to (149.4, 118.8)
- moved J6 1.28 mm to (148.2, 120.8)
- moved C16 1.25 mm to (65.1, 149.4)
- moved C17 1.25 mm to (67.1, 149.4)
- moved C18 1.25 mm to (69.1, 149.4)
- moved C21 1.25 mm to (65.1, 153.4)
- moved C22 1.25 mm to (67.1, 153.4)
- moved C23 1.25 mm to (69.1, 153.4)
- moved C14 1.25 mm to (61.1, 149.4)
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Routing:
- net /OUT_DC2-: track 37.5 -> 47.6 mm, vias 1 -> 2
- net /LS_HOT1: track 143.7 -> 137.5 mm
- net +3.3V: track 108.0 -> 105.7 mm
- net /DC2_DIR: track 73.7 -> 71.5 mm
- net /LS_HOT2: track 141.8 -> 139.6 mm
- net +5VA: track 172.3 -> 170.3 mm
- net Net-(U6-IN2): track 2.89 -> 4.49 mm
- net /CAN+: track 101.7 -> 103.0 mm
- net /5_WBO_Rtrim: track 13.5 -> 12.2 mm
- net /6_WBO_Un: track 23.4 -> 22.1 mm
- net /2_WBO_Vm: track 17.2 -> 15.9 mm
- net /1_WBO_Ip: track 18.2 -> 16.9 mm
- net /3_WBO_Heater: track 8.54 -> 7.27 mm
- net Net-(M6-UART2_RX_(PD6)): track 67.5 -> 66.3 mm
- net /CAN-: track 101.1 -> 102.2 mm
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