File: INJ6.kicad_sch (KiCad schematic)
At the start: 12 parts, among them Q10 ZXMS6005SGTA, Q11 ZXMS6005SGTA, Q13 ZXMS6005SGTA, Q7 ZXMS6005SGTA, Q8 ZXMS6005SGTA, Q9 ZXMS6005SGTA

Commit message: Upd SCH
Parts:
- renumbered Q7 to Q14, Q8 to Q15, Q9 to Q16, Q10 to Q17, Q11 to Q18
Changed lines of the file:
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@@
   (symbol (lib_id "Transistor_FET:BSP129") (at 165.1 66.04 0) (mirror y) (unit 1)
     (in_bom yes) (on_board yes) (dnp no) (fields_autoplaced)
-    (property "Reference" "Q9" (at 158.75 64.77 0)
+    (property "Reference" "Q16" (at 158.75 64.77 0)
       (effects (font (size 1.27 1.27)) (justify left))
     )
@@
       (project "uaefi"
         (path "/ac264c30-3e9a-4be2-b97a-9949b68bd497/45207479-6ae5-486c-ab42-805dda4ce511"
-          (reference "Q9") (unit 1)
+          (reference "Q16") (unit 1)
         )
         (path "/ac264c30-3e9a-4be2-b97a-9949b68bd497/aa4a40ff-b05c-4d24-92a7-fdeac4807f5c"
@@
         )
         (path "/ac264c30-3e9a-4be2-b97a-9949b68bd497/45207479-6ae5-486c-ab42-805dda4ce511"
-          (reference "#PWR09") (unit 1)
+          (reference "#PWR0112") (unit 1)
         )
         (path "/ac264c30-3e9a-4be2-b97a-9949b68bd497/aa4a40ff-b05c-4d24-92a7-fdeac4807f5c"
@@
         )
         (path "/ac264c30-3e9a-4be2-b97a-9949b68bd497/45207479-6ae5-486c-ab42-805dda4ce511"
-          (reference "#PWR014") (unit 1)
+          (reference "#PWR0114") (unit 1)
         )
         (path "/ac264c30-3e9a-4be2-b97a-9949b68bd497/aa4a40ff-b05c-4d24-92a7-fdeac4807f5c"
@@
   (symbol (lib_id "Transistor_FET:BSP129") (at 118.11 121.92 0) (mirror y) (unit 1)
     (in_bom yes) (on_board yes) (dnp no) (fields_autoplaced)
-    (property "Reference" "Q8" (at 111.76 120.65 0)
+    (property "Reference" "Q15" (at 111.76 120.65 0)
       (effects (font (size 1.27 1.27)) (justify left))
     )
@@
       (project "uaefi"
         (path "/ac264c30-3e9a-4be2-b97a-9949b68bd497/45207479-6ae5-486c-ab42-805dda4ce511"
-          (reference "Q8") (unit 1)
+          (reference "Q15") (unit 1)
         )
         (path "/ac264c30-3e9a-4be2-b97a-9949b68bd497/aa4a40ff-b05c-4d24-92a7-fdeac4807f5c"
@@
         )
         (path "/ac264c30-3e9a-4be2-b97a-9949b68bd497/45207479-6ae5-486c-ab42-805dda4ce511"
-          (reference "R32") (unit 1)
+          (reference "R31") (unit 1)
         )
         (path "/ac264c30-3e9a-4be2-b97a-9949b68bd497/aa4a40ff-b05c-4d24-92a7-fdeac4807f5c"
@@
         )
         (path "/ac264c30-3e9a-4be2-b97a-9949b68bd497/45207479-6ae5-486c-ab42-805dda4ce511"
-          (reference "#PWR08") (unit 1)
+          (reference "#PWR0111") (unit 1)
         )
         (path "/ac264c30-3e9a-4be2-b97a-9949b68bd497/aa4a40ff-b05c-4d24-92a7-fdeac4807f5c"
@@
   (symbol (lib_id "Transistor_FET:BSP129") (at 118.11 93.98 0) (mirror y) (unit 1)
     (in_bom yes) (on_board yes) (dnp no) (fields_autoplaced)
-    (property "Reference" "Q7" (at 111.76 92.71 0)
+    (property "Reference" "Q14" (at 111.76 92.71 0)
       (effects (font (size 1.27 1.27)) (justify left))
     )
@@
       (project "uaefi"
         (path "/ac264c30-3e9a-4be2-b97a-9949b68bd497/45207479-6ae5-486c-ab42-805dda4ce511"
-          (reference "Q7") (unit 1)
+          (reference "Q14") (unit 1)
         )
         (path "/ac264c30-3e9a-4be2-b97a-9949b68bd497/aa4a40ff-b05c-4d24-92a7-fdeac4807f5c"
@@
         )
         (path "/ac264c30-3e9a-4be2-b97a-9949b68bd497/45207479-6ae5-486c-ab42-805dda4ce511"
-          (reference "#PWR015") (unit 1)
+          (reference "#PWR0115") (unit 1)
         )
         (path "/ac264c30-3e9a-4be2-b97a-9949b68bd497/aa4a40ff-b05c-4d24-92a7-fdeac4807f5c"
@@
         )
         (path "/ac264c30-3e9a-4be2-b97a-9949b68bd497/45207479-6ae5-486c-ab42-805dda4ce511"
-          (reference "#PWR013") (unit 1)
+          (reference "#PWR0113") (unit 1)
         )
         (path "/ac264c30-3e9a-4be2-b97a-9949b68bd497/aa4a40ff-b05c-4d24-92a7-fdeac4807f5c"
@@
   (symbol (lib_id "Transistor_FET:BSP129") (at 165.1 121.92 0) (mirror y) (unit 1)
     (in_bom yes) (on_board yes) (dnp no) (fields_autoplaced)
-    (property "Reference" "Q11" (at 158.75 120.65 0)
+    (property "Reference" "Q18" (at 158.75 120.65 0)
       (effects (font (size 1.27 1.27)) (justify left))
     )
@@
       (project "uaefi"
         (path "/ac264c30-3e9a-4be2-b97a-9949b68bd497/45207479-6ae5-486c-ab42-805dda4ce511"
-          (reference "Q11") (unit 1)
+          (reference "Q18") (unit 1)
         )
         (path "/ac264c30-3e9a-4be2-b97a-9949b68bd497/aa4a40ff-b05c-4d24-92a7-fdeac4807f5c"
@@
         )
         (path "/ac264c30-3e9a-4be2-b97a-9949b68bd497/45207479-6ae5-486c-ab42-805dda4ce511"
-          (reference "R35") (unit 1)
+          (reference "R34") (unit 1)
         )
         (path "/ac264c30-3e9a-4be2-b97a-9949b68bd497/aa4a40ff-b05c-4d24-92a7-fdeac4807f5c"
@@
   (symbol (lib_id "Transistor_FET:BSP129") (at 165.1 93.98 0) (mirror y) (unit 1)
     (in_bom yes) (on_board yes) (dnp no) (fields_autoplaced)
-    (property "Reference" "Q10" (at 158.75 92.71 0)
+    (property "Reference" "Q17" (at 158.75 92.71 0)
       (effects (font (size 1.27 1.27)) (justify left))
     )
@@
       (project "uaefi"
         (path "/ac264c30-3e9a-4be2-b97a-9949b68bd497/45207479-6ae5-486c-ab42-805dda4ce511"
-          (reference "Q10") (unit 1)
+          (reference "Q17") (unit 1)
         )
         (path "/ac264c30-3e9a-4be2-b97a-9949b68bd497/aa4a40ff-b05c-4d24-92a7-fdeac4807f5c"
@@
         )
         (path "/ac264c30-3e9a-4be2-b97a-9949b68bd497/45207479-6ae5-486c-ab42-805dda4ce511"
-          (reference "#PWR016") (unit 1)
+          (reference "#PWR0116") (unit 1)
         )
         (path "/ac264c30-3e9a-4be2-b97a-9949b68bd497/aa4a40ff-b05c-4d24-92a7-fdeac4807f5c"
@@
         )
         (path "/ac264c30-3e9a-4be2-b97a-9949b68bd497/45207479-6ae5-486c-ab42-805dda4ce511"
-          (reference "R31") (unit 1)
+          (reference "R30") (unit 1)
         )
         (path "/ac264c30-3e9a-4be2-b97a-9949b68bd497/aa4a40ff-b05c-4d24-92a7-fdeac4807f5c"
@@
         )
         (path "/ac264c30-3e9a-4be2-b97a-9949b68bd497/45207479-6ae5-486c-ab42-805dda4ce511"
-          (reference "R34") (unit 1)
+          (reference "R33") (unit 1)
         )
         (path "/ac264c30-3e9a-4be2-b97a-9949b68bd497/aa4a40ff-b05c-4d24-92a7-fdeac4807f5c"
@@
         )
         (path "/ac264c30-3e9a-4be2-b97a-9949b68bd497/45207479-6ae5-486c-ab42-805dda4ce511"
-          (reference "R33") (unit 1)
+          (reference "R32") (unit 1)
         )
         (path "/ac264c30-3e9a-4be2-b97a-9949b68bd497/aa4a40ff-b05c-4d24-92a7-fdeac4807f5c"
@@
         )
         (path "/ac264c30-3e9a-4be2-b97a-9949b68bd497/45207479-6ae5-486c-ab42-805dda4ce511"
-          (reference "R30") (unit 1)
-        )
-        (path "/ac264c30-3e9a-4be2-b97a-9949b68bd497/aa4a40ff-b05c-4d24-92a7-fdeac4807f5c"
+          (reference "R29") (unit 1)
+        )
+        (path "/ac264c30-3e9a-4be2-b97a-9949b68bd497/aa4a40ff-b05c-4d24-92a7-fdeac4807f5c"

Commit message: Upd SCH, PCB
Parts:
- removed Q13, Q14, Q15, Q16, Q17, Q18: ZXMS6005SGTA, Package_TO_SOT_SMD:SOT-223, symbol Transistor_FET:BSP129
- added U10, U11, U9: VNLD5160TR-E, Package_SO:SOIC-8_3.9x4.9mm_P1.27mm, symbol chips:VNLD5160
Connections:
- net GND: now also U10.5 (S2), U10.7 (S1), U11.5 (S2), U11.7 (S1), U9.5 (S2), U9.7 (S1)
- net IN1: now also U9.1 (IN1)
- net IN2: now also U9.3 (IN2)
- net IN3: now also U10.1 (IN1)
- net IN4: now also U10.3 (IN2)
- net IN5: now also U11.1 (IN1)
- net IN6: now also U11.3 (IN2)
- net OUT1: now also U9.8 (D1)
- net OUT2: now also U9.6 (D2)
- net OUT3: now also U10.8 (D1)
- net OUT4: now also U10.6 (D2)
- net OUT5: now also U11.8 (D1)
- net OUT6: now also U11.6 (D2)
- no-connect marks 0 -> 6
Other:
- moved on the sheet: R30
