File: INJ6.kicad_sch (KiCad schematic)
At the start: 9 parts, among them U10 VNLD5160TR-E, U11 VNLD5160TR-E, U9 VNLD5160TR-E

Commit message: #66
Other:
- company: rusefi.com -> rusEFI.com
- title: UAEFI Injector -> UAEFI
