File: LS4.kicad_sch (KiCad schematic)
At the start: 12 parts, among them Q13 ZXMS6005SGTA, Q7 ZXMS6005SGTA, Q8 ZXMS6005SGTA, Q9 ZXMS6005SGTA

Commit message: Upd PCB
Parts:
- renumbered Q13 to Q1, Q7 to Q2, Q8 to Q3, Q9 to Q4
Changed lines of the file:
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@@
   (symbol (lib_id "Transistor_FET:BSP129") (at 162.56 66.04 0) (mirror y) (unit 1)
     (in_bom yes) (on_board yes) (dnp no) (fields_autoplaced)
-    (property "Reference" "Q8" (at 156.21 64.77 0)
+    (property "Reference" "Q3" (at 156.21 64.77 0)
       (effects (font (size 1.27 1.27)) (justify left))
     )
@@
     (instances
       (project "uaefi"
-        (path "/ac264c30-3e9a-4be2-b97a-9949b68bd497/45207479-6ae5-486c-ab42-805dda4ce511"
-          (reference "Q8") (unit 1)
-        )
         (path "/ac264c30-3e9a-4be2-b97a-9949b68bd497/aa4a40ff-b05c-4d24-92a7-fdeac4807f5c"
           (reference "Q3") (unit 1)
@@
       )
       (project "uaefi"
-        (path "/ac264c30-3e9a-4be2-b97a-9949b68bd497"
-          (reference "#PWR022") (unit 1)
-        )
         (path "/ac264c30-3e9a-4be2-b97a-9949b68bd497/aa4a40ff-b05c-4d24-92a7-fdeac4807f5c"
           (reference "#PWR074") (unit 1)
@@
       )
       (project "uaefi"
-        (path "/ac264c30-3e9a-4be2-b97a-9949b68bd497"
-          (reference "R53") (unit 1)
-        )
-        (path "/ac264c30-3e9a-4be2-b97a-9949b68bd497/45207479-6ae5-486c-ab42-805dda4ce511"
-          (reference "R30") (unit 1)
-        )
         (path "/ac264c30-3e9a-4be2-b97a-9949b68bd497/aa4a40ff-b05c-4d24-92a7-fdeac4807f5c"
           (reference "R10") (unit 1)
@@
       )
       (project "uaefi"
-        (path "/ac264c30-3e9a-4be2-b97a-9949b68bd497"
-          (reference "#PWR022") (unit 1)
-        )
         (path "/ac264c30-3e9a-4be2-b97a-9949b68bd497/aa4a40ff-b05c-4d24-92a7-fdeac4807f5c"
           (reference "#PWR070") (unit 1)
@@
       )
       (project "uaefi"
-        (path "/ac264c30-3e9a-4be2-b97a-9949b68bd497"
-          (reference "#PWR018") (unit 1)
-        )
-        (path "/ac264c30-3e9a-4be2-b97a-9949b68bd497/92c4206f-a69e-4d4d-9308-206d3518e11e"
-          (reference "#PWR02") (unit 1)
-        )
-        (path "/ac264c30-3e9a-4be2-b97a-9949b68bd497/45207479-6ae5-486c-ab42-805dda4ce511"
-          (reference "#PWR09") (unit 1)
-        )
         (path "/ac264c30-3e9a-4be2-b97a-9949b68bd497/aa4a40ff-b05c-4d24-92a7-fdeac4807f5c"
           (reference "#PWR068") (unit 1)
@@
       )
       (project "uaefi"
-        (path "/ac264c30-3e9a-4be2-b97a-9949b68bd497"
-          (reference "R53") (unit 1)
-        )
-        (path "/ac264c30-3e9a-4be2-b97a-9949b68bd497/45207479-6ae5-486c-ab42-805dda4ce511"
-          (reference "R32") (unit 1)
-        )
         (path "/ac264c30-3e9a-4be2-b97a-9949b68bd497/aa4a40ff-b05c-4d24-92a7-fdeac4807f5c"
           (reference "R12") (unit 1)
@@
   (symbol (lib_id "Transistor_FET:BSP129") (at 115.57 93.98 0) (mirror y) (unit 1)
     (in_bom yes) (on_board yes) (dnp no) (fields_autoplaced)
-    (property "Reference" "Q7" (at 109.22 92.71 0)
+    (property "Reference" "Q2" (at 109.22 92.71 0)
       (effects (font (size 1.27 1.27)) (justify left))
     )
@@
     (instances
       (project "uaefi"
-        (path "/ac264c30-3e9a-4be2-b97a-9949b68bd497/45207479-6ae5-486c-ab42-805dda4ce511"
-          (reference "Q7") (unit 1)
-        )
         (path "/ac264c30-3e9a-4be2-b97a-9949b68bd497/aa4a40ff-b05c-4d24-92a7-fdeac4807f5c"
           (reference "Q2") (unit 1)
@@
   (symbol (lib_id "Transistor_FET:BSP129") (at 115.57 66.04 0) (mirror y) (unit 1)
     (in_bom yes) (on_board yes) (dnp no) (fields_autoplaced)
-    (property "Reference" "Q13" (at 109.22 64.77 0)
+    (property "Reference" "Q1" (at 109.22 64.77 0)
       (effects (font (size 1.27 1.27)) (justify left))
     )
@@
     (instances
       (project "uaefi"
-        (path "/ac264c30-3e9a-4be2-b97a-9949b68bd497/45207479-6ae5-486c-ab42-805dda4ce511"
-          (reference "Q13") (unit 1)
-        )
         (path "/ac264c30-3e9a-4be2-b97a-9949b68bd497/aa4a40ff-b05c-4d24-92a7-fdeac4807f5c"
           (reference "Q1") (unit 1)
@@
       )
       (project "uaefi"
-        (path "/ac264c30-3e9a-4be2-b97a-9949b68bd497"
-          (reference "D12") (unit 1)
-        )
         (path "/ac264c30-3e9a-4be2-b97a-9949b68bd497/aa4a40ff-b05c-4d24-92a7-fdeac4807f5c"
           (reference "D5") (unit 1)
@@
       )
       (project "uaefi"
-        (path "/ac264c30-3e9a-4be2-b97a-9949b68bd497"
-          (reference "#PWR018") (unit 1)
-        )
-        (path "/ac264c30-3e9a-4be2-b97a-9949b68bd497/92c4206f-a69e-4d4d-9308-206d3518e11e"
-          (reference "#PWR02") (unit 1)
-        )
-        (path "/ac264c30-3e9a-4be2-b97a-9949b68bd497/45207479-6ae5-486c-ab42-805dda4ce511"
-          (reference "#PWR013") (unit 1)
-        )
         (path "/ac264c30-3e9a-4be2-b97a-9949b68bd497/aa4a40ff-b05c-4d24-92a7-fdeac4807f5c"
           (reference "#PWR071") (unit 1)
@@
       )
       (project "uaefi"
-        (path "/ac264c30-3e9a-4be2-b97a-9949b68bd497"
-          (reference "#PWR022") (unit 1)
-        )
         (path "/ac264c30-3e9a-4be2-b97a-9949b68bd497/aa4a40ff-b05c-4d24-92a7-fdeac4807f5c"
           (reference "#PWR069") (unit 1)
@@
       )
       (project "uaefi"
-        (path "/ac264c30-3e9a-4be2-b97a-9949b68bd497"
-          (reference "#PWR022") (unit 1)
-        )
         (path "/ac264c30-3e9a-4be2-b97a-9949b68bd497/aa4a40ff-b05c-4d24-92a7-fdeac4807f5c"
           (reference "#PWR073") (unit 1)
@@
       )
       (project "uaefi"
-        (path "/ac264c30-3e9a-4be2-b97a-9949b68bd497"
-          (reference "D12") (unit 1)
-        )
         (path "/ac264c30-3e9a-4be2-b97a-9949b68bd497/aa4a40ff-b05c-4d24-92a7-fdeac4807f5c"
           (reference "D4") (unit 1)
@@
   (symbol (lib_id "Transistor_FET:BSP129") (at 162.56 93.98 0) (mirror y) (unit 1)
     (in_bom yes) (on_board yes) (dnp no) (fields_autoplaced)
-    (property "Reference" "Q9" (at 156.21 92.71 0)
+    (property "Reference" "Q4" (at 156.21 92.71 0)
       (effects (font (size 1.27 1.27)) (justify left))
     )
@@
     (instances
       (project "uaefi"
-        (path "/ac264c30-3e9a-4be2-b97a-9949b68bd497/45207479-6ae5-486c-ab42-805dda4ce511"
-          (reference "Q9") (unit 1)
-        )
         (path "/ac264c30-3e9a-4be2-b97a-9949b68bd497/aa4a40ff-b05c-4d24-92a7-fdeac4807f5c"
           (reference "Q4") (unit 1)
@@
       )
       (project "uaefi"
-        (path "/ac264c30-3e9a-4be2-b97a-9949b68bd497"
-          (reference "#PWR018") (unit 1)
-        )
-        (path "/ac264c30-3e9a-4be2-b97a-9949b68bd497/92c4206f-a69e-4d4d-9308-206d3518e11e"
-          (reference "#PWR02") (unit 1)
-        )
-        (path "/ac264c30-3e9a-4be2-b97a-9949b68bd497/45207479-6ae5-486c-ab42-805dda4ce511"
-          (reference "#PWR08") (unit 1)
-        )
         (path "/ac264c30-3e9a-4be2-b97a-9949b68bd497/aa4a40ff-b05c-4d24-92a7-fdeac4807f5c"
           (reference "#PWR067") (unit 1)
@@
       )
       (project "uaefi"
-        (path "/ac264c30-3e9a-4be2-b97a-9949b68bd497"
-          (reference "D12") (unit 1)
-        )
         (path "/ac264c30-3e9a-4be2-b97a-9949b68bd497/aa4a40ff-b05c-4d24-92a7-fdeac4807f5c"
           (reference "D2") (unit 1)
@@
       )
       (project "uaefi"
-        (path "/ac264c30-3e9a-4be2-b97a-9949b68bd497"
-          (reference "#PWR018") (unit 1)
-        )
-        (path "/ac264c30-3e9a-4be2-b97a-9949b68bd497/92c4206f-a69e-4d4d-9308-206d3518e11e"
-          (reference "#PWR02") (unit 1)
-        )
-        (path "/ac264c30-3e9a-4be2-b97a-9949b68bd497/45207479-6ae5-486c-ab42-805dda4ce511"
-          (reference "#PWR014") (unit 1)
-        )
         (path "/ac264c30-3e9a-4be2-b97a-9949b68bd497/aa4a40ff-b05c-4d24-92a7-fdeac4807f5c"
           (reference "#PWR072") (unit 1)
@@
       )
       (project "uaefi"
-        (path "/ac264c30-3e9a-4be2-b97a-9949b68bd497"
-          (reference "D12") (unit 1)
-        )
         (path "/ac264c30-3e9a-4be2-b97a-9949b68bd497/aa4a40ff-b05c-4d24-92a7-fdeac4807f5c"
           (reference "D3") (unit 1)
@@
       )
       (project "uaefi"
-        (path "/ac264c30-3e9a-4be2-b97a-9949b68bd497"
-          (reference "R53") (unit 1)
-        )
-        (path "/ac264c30-3e9a-4be2-b97a-9949b68bd497/45207479-6ae5-486c-ab42-805dda4ce511"
-          (reference "R33") (unit 1)
-        )
         (path "/ac264c30-3e9a-4be2-b97a-9949b68bd497/aa4a40ff-b05c-4d24-92a7-fdeac4807f5c"
           (reference "R13") (unit 1)
@@
       )
       (project "uaefi"
-        (path "/ac264c30-3e9a-4be2-b97a-9949b68bd497"
-          (reference "R53") (unit 1)
-        )
-        (path "/ac264c30-3e9a-4be2-b97a-9949b68bd497/45207479-6ae5-486c-ab42-805dda4ce511"
-          (reference "R31") (unit 1)
-        )
         (path "/ac264c30-3e9a-4be2-b97a-9949b68bd497/aa4a40ff-b05c-4d24-92a7-fdeac4807f5c"
           (reference "R11") (unit 1)

Commit message: Upd SCH, PCB
Parts:
- removed Q1, Q2, Q3, Q4: ZXMS6005SGTA, Package_TO_SOT_SMD:SOT-223, symbol Transistor_FET:BSP129
- added U7, U8: VNLD5160TR-E, Package_SO:SOIC-8_3.9x4.9mm_P1.27mm, symbol chips:VNLD5160
Connections:
- net GND: now also U7.5 (S2), U7.7 (S1), U8.5 (S2), U8.7 (S1)
- net IN1: now also U7.1 (IN1)
- net IN2: now also U7.3 (IN2)
- net IN3: now also U8.1 (IN1)
- net IN4: now also U8.3 (IN2)
- net OUT1: now also U7.8 (D1)
- net OUT2: now also U7.6 (D2)
- net OUT3: now also U8.8 (D1)
- net OUT4: now also U8.6 (D2)
- no-connect marks 0 -> 4
Other:
- moved on the sheet: D27, R30
