File: LS4.kicad_sch (KiCad schematic)
At the start: 10 parts, among them U7 VNLD5160TR-E, U8 VNLD5160TR-E

Commit message: #66
Other:
- company: rusefi.com -> rusEFI.com
- title: UAEFI Low Side -> UAEFI

Commit message: #81 #82 #86 #87
Parts:
- removed D27 (x4): B5819W, hellen-one-common:SOD-123, symbol hellen-one-common:1N4148WS
