File: egt.kicad_sch (KiCad schematic)
At the start: 9 parts, among them U1 MAX31855KASA

Commit message: Upd SCH
Parts:
- renumbered C48 to C28, C49 to C29, C27 to C30, C37 to C31, C43 to C32, D7 to D8, L3 to L2, U1 to U4
Changed lines of the file:
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@@
   (symbol (lib_id "Device:C") (at 154.94 101.6 0) (mirror y) (unit 1)
     (in_bom no) (on_board yes) (dnp no)
-    (property "Reference" "C27" (at 152.019 100.4316 0)
+    (property "Reference" "C30" (at 152.019 100.4316 0)
       (effects (font (size 1.27 1.27)) (justify left))
     )
@@
       (project "uaefi"
         (path "/ac264c30-3e9a-4be2-b97a-9949b68bd497/ced20183-e5c8-42b4-80bd-35fc70d9313a"
-          (reference "C27") (unit 1)
+          (reference "C30") (unit 1)
         )
       )
@@
   (symbol (lib_id "Power_Protection:NUP2105L") (at 119.38 101.6 0) (mirror y) (unit 1)
     (in_bom yes) (on_board yes) (dnp no)
-    (property "Reference" "D7" (at 114.3 106.68 0)
+    (property "Reference" "D8" (at 114.3 106.68 0)
       (effects (font (size 1.27 1.27)) (justify left))
     )
@@
       (project "uaefi"
         (path "/ac264c30-3e9a-4be2-b97a-9949b68bd497/ced20183-e5c8-42b4-80bd-35fc70d9313a"
-          (reference "D7") (unit 1)
+          (reference "D8") (unit 1)
         )
       )
@@
   (symbol (lib_id "Sensor_Temperature:MAX31855KASA") (at 166.37 92.71 0) (unit 1)
     (in_bom yes) (on_board yes) (dnp no) (fields_autoplaced)
-    (property "Reference" "U1" (at 168.3894 80.01 0)
+    (property "Reference" "U4" (at 168.3894 80.01 0)
       (effects (font (size 1.27 1.27)) (justify left))
     )
@@
       (project "uaefi"
         (path "/ac264c30-3e9a-4be2-b97a-9949b68bd497/ced20183-e5c8-42b4-80bd-35fc70d9313a"
-          (reference "U1") (unit 1)
+          (reference "U4") (unit 1)
         )
       )
@@
   (symbol (lib_name "GND_4") (lib_id "power:GND") (at 176.53 77.47 0) (unit 1)
     (in_bom yes) (on_board yes) (dnp no)
-    (property "Reference" "#PWR0150" (at 176.53 83.82 0)
+    (property "Reference" "#PWR0109" (at 176.53 83.82 0)
       (effects (font (size 1.27 1.27)) hide)
     )
@@
       (project "uaefi"
         (path "/ac264c30-3e9a-4be2-b97a-9949b68bd497/ced20183-e5c8-42b4-80bd-35fc70d9313a"
-          (reference "#PWR0150") (unit 1)
+          (reference "#PWR0109") (unit 1)
         )
       )
@@
   (symbol (lib_id "Device:L") (at 106.68 95.25 90) (unit 1)
     (in_bom yes) (on_board yes) (dnp no)
-    (property "Reference" "L3" (at 106.68 97.79 90)
+    (property "Reference" "L2" (at 106.68 97.79 90)
       (effects (font (size 1.27 1.27)))
     )
@@
       (project "uaefi"
         (path "/ac264c30-3e9a-4be2-b97a-9949b68bd497/ced20183-e5c8-42b4-80bd-35fc70d9313a"
-          (reference "L3") (unit 1)
+          (reference "L2") (unit 1)
         )
       )
@@
   (symbol (lib_name "GND_3") (lib_id "power:GND") (at 189.23 77.47 0) (unit 1)
     (in_bom yes) (on_board yes) (dnp no)
-    (property "Reference" "#PWR0149" (at 189.23 83.82 0)
+    (property "Reference" "#PWR0110" (at 189.23 83.82 0)
       (effects (font (size 1.27 1.27)) hide)
     )
@@
       (project "uaefi"
         (path "/ac264c30-3e9a-4be2-b97a-9949b68bd497/ced20183-e5c8-42b4-80bd-35fc70d9313a"
-          (reference "#PWR0149") (unit 1)
+          (reference "#PWR0110") (unit 1)
         )
       )
@@
   (symbol (lib_name "GND_5") (lib_id "power:GND") (at 139.7 107.95 0) (unit 1)
     (in_bom yes) (on_board yes) (dnp no)
-    (property "Reference" "#PWR0156" (at 139.7 114.3 0)
+    (property "Reference" "#PWR0106" (at 139.7 114.3 0)
       (effects (font (size 1.27 1.27)) hide)
     )
@@
       (project "uaefi"
         (path "/ac264c30-3e9a-4be2-b97a-9949b68bd497/ced20183-e5c8-42b4-80bd-35fc70d9313a"
-          (reference "#PWR0156") (unit 1)
+          (reference "#PWR0106") (unit 1)
         )
       )
@@
   (symbol (lib_name "GND_6") (lib_id "power:GND") (at 154.94 107.95 0) (unit 1)
     (in_bom yes) (on_board yes) (dnp no)
-    (property "Reference" "#PWR0157" (at 154.94 114.3 0)
+    (property "Reference" "#PWR0107" (at 154.94 114.3 0)
       (effects (font (size 1.27 1.27)) hide)
     )
@@
       (project "uaefi"
         (path "/ac264c30-3e9a-4be2-b97a-9949b68bd497/ced20183-e5c8-42b4-80bd-35fc70d9313a"
-          (reference "#PWR0157") (unit 1)
+          (reference "#PWR0107") (unit 1)
         )
       )
@@
   (symbol (lib_name "GND_7") (lib_id "power:GND") (at 166.37 105.41 0) (unit 1)
     (in_bom yes) (on_board yes) (dnp no)
-    (property "Reference" "#PWR0148" (at 166.37 111.76 0)
+    (property "Reference" "#PWR0108" (at 166.37 111.76 0)
       (effects (font (size 1.27 1.27)) hide)
     )
@@
       (project "uaefi"
         (path "/ac264c30-3e9a-4be2-b97a-9949b68bd497/ced20183-e5c8-42b4-80bd-35fc70d9313a"
-          (reference "#PWR0148") (unit 1)
+          (reference "#PWR0108") (unit 1)
         )
       )
@@
   (symbol (lib_id "Device:C") (at 147.32 91.44 180) (unit 1)
     (in_bom yes) (on_board yes) (dnp no)
-    (property "Reference" "C49" (at 144.399 92.6084 0)
+    (property "Reference" "C29" (at 144.399 92.6084 0)
       (effects (font (size 1.27 1.27)) (justify left))
     )
@@
       (project "uaefi"
         (path "/ac264c30-3e9a-4be2-b97a-9949b68bd497/ced20183-e5c8-42b4-80bd-35fc70d9313a"
-          (reference "C49") (unit 1)
+          (reference "C29") (unit 1)
         )
       )
@@
   (symbol (lib_id "Device:C") (at 139.7 101.6 0) (mirror y) (unit 1)
     (in_bom no) (on_board yes) (dnp no)
-    (property "Reference" "C48" (at 136.779 100.4316 0)
+    (property "Reference" "C28" (at 136.779 100.4316 0)
       (effects (font (size 1.27 1.27)) (justify left))
     )
@@
       (project "uaefi"
         (path "/ac264c30-3e9a-4be2-b97a-9949b68bd497/ced20183-e5c8-42b4-80bd-35fc70d9313a"
-          (reference "C48") (unit 1)
+          (reference "C28") (unit 1)
         )
       )
@@
   (symbol (lib_id "Device:C") (at 189.23 73.66 0) (unit 1)
     (in_bom yes) (on_board yes) (dnp no)
-    (property "Reference" "C43" (at 192.151 72.4916 0)
+    (property "Reference" "C32" (at 192.151 72.4916 0)
       (effects (font (size 1.27 1.27)) (justify left))
     )
@@
       (project "uaefi"
         (path "/ac264c30-3e9a-4be2-b97a-9949b68bd497/ced20183-e5c8-42b4-80bd-35fc70d9313a"
-          (reference "C43") (unit 1)
+          (reference "C32") (unit 1)
         )
       )
@@
   (symbol (lib_id "power:GND") (at 119.38 107.95 0) (unit 1)
     (in_bom yes) (on_board yes) (dnp no)
-    (property "Reference" "#PWR0154" (at 119.38 114.3 0)
+    (property "Reference" "#PWR0105" (at 119.38 114.3 0)
       (effects (font (size 1.27 1.27)) hide)
     )
@@
       (project "uaefi"
         (path "/ac264c30-3e9a-4be2-b97a-9949b68bd497/ced20183-e5c8-42b4-80bd-35fc70d9313a"
-          (reference "#PWR0154") (unit 1)
+          (reference "#PWR0105") (unit 1)
         )
       )
@@
   (symbol (lib_id "Device:C") (at 176.53 73.66 0) (unit 1)
     (in_bom yes) (on_board yes) (dnp no)
-    (property "Reference" "C37" (at 179.451 72.4916 0)
+    (property "Reference" "C31" (at 179.451 72.4916 0)
       (effects (font (size 1.27 1.27)) (justify left))
     )
@@
       (project "uaefi"
         (path "/ac264c30-3e9a-4be2-b97a-9949b68bd497/ced20183-e5c8-42b4-80bd-35fc70d9313a"
-          (reference "C37") (unit 1)
-        )
-      )
+          (reference "C31") (unit 1)
+        )
+      )

Commit message: Placement
Changed lines of the file:
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@@
     (effects (font (size 1.27 1.27)) (justify right))
   )
-  (symbol (lib_id "Device:C") (at 154.94 101.6 0) (mirror y) (unit 1)
-    (in_bom no) (on_board yes) (dnp no)
-    (property "Reference" "C30" (at 152.019 100.4316 0)
-      (effects (font (size 1.27 1.27)) (justify left))
-    )
-    (property "Value" "10nF 50V" (at 152.019 102.743 0)
-      (effects (font (size 1.27 1.27)) (justify left))
-    )
-    (property "Footprint" "Capacitor_SMD:C_0402_1005Metric" (at 153.9748 105.41 0)
-      (effects (font (size 1.27 1.27)) hide)
-    )
-    (property "Datasheet" "~" (at 154.94 101.6 0)
-      (effects (font (size 1.27 1.27)) hide)
-    )
-    (property "LCSC" "" (at 154.94 101.6 0)
-      (effects (font (size 1.27 1.27)) hide)
-    )
-    (property "MyComment" "DNP" (at 149.86 105.41 0)
-      (effects (font (size 1.27 1.27)))
-    )
-    (pin "1")
-    (pin "2")
-    (instances
-      (project "uaefi"
-        (path "/ac264c30-3e9a-4be2-b97a-9949b68bd497/ced20183-e5c8-42b4-80bd-35fc70d9313a"
-          (reference "C30") (unit 1)
-        )
-      )
-    )
-  )
-  (symbol (lib_id "Power_Protection:NUP2105L") (at 119.38 101.6 0) (mirror y) (unit 1)
-    (in_bom yes) (on_board yes) (dnp no)
-    (property "Reference" "D8" (at 114.3 106.68 0)
-      (effects (font (size 1.27 1.27)) (justify left))
-    )
-    (property "Value" "NUP2105L" (at 114.3 109.22 0)
-      (effects (font (size 1.27 1.27)) (justify left))
-    )
-    (property "Footprint" "Package_TO_SOT_SMD:SOT-23" (at 113.665 102.87 0)
-      (effects (font (size 1.27 1.27)) (justify left) hide)
-    )
-    (property "Datasheet" "http://www.onsemi.com/pub_link/Collateral/NUP2105L-D.PDF" (at 116.205 98.425 0)
-      (effects (font (size 1.27 1.27)) hide)
-    )
-    (property "LCSC" "C284104" (at 119.38 101.6 0)
-      (effects (font (size 1.27 1.27)) hide)
-    )
-    (pin "3")
-    (pin "1")
-    (pin "2")
-    (instances
-      (project "uaefi"
-        (path "/ac264c30-3e9a-4be2-b97a-9949b68bd497/ced20183-e5c8-42b4-80bd-35fc70d9313a"
-          (reference "D8") (unit 1)
-        )
-      )
-    )
-  )
-  (symbol (lib_id "Sensor_Temperature:MAX31855KASA") (at 166.37 92.71 0) (unit 1)
+  (symbol (lib_name "MAX31855KASA_1") (lib_id "Sensor_Temperature:MAX31855KASA") (at 166.37 92.71 0) (unit 1)
     (in_bom yes) (on_board yes) (dnp no) (fields_autoplaced)
-    (property "Reference" "U4" (at 168.3894 80.01 0)
-      (effects (font (size 1.27 1.27)) (justify left))
-    )
-    (property "Value" "MAX31855KASA" (at 168.3894 82.55 0)
+    (property "Reference" "U4" (at 168.5641 80.01 0)
+      (effects (font (size 1.27 1.27)) (justify left))
+    )
+    (property "Value" "MAX31855KASA" (at 168.5641 82.55 0)
       (effects (font (size 1.27 1.27)) (justify left))
     )
@@
     )
   )
+  (symbol (lib_id "Device:C") (at 154.94 101.6 0) (mirror y) (unit 1)
+    (in_bom no) (on_board yes) (dnp no)
+    (property "Reference" "C30" (at 152.019 100.4316 0)
+      (effects (font (size 1.27 1.27)) (justify left))
+    )
+    (property "Value" "10nF 50V" (at 152.019 102.743 0)
+      (effects (font (size 1.27 1.27)) (justify left))
+    )
+    (property "Footprint" "Capacitor_SMD:C_0402_1005Metric" (at 153.9748 105.41 0)
+      (effects (font (size 1.27 1.27)) hide)
+    )
+    (property "Datasheet" "~" (at 154.94 101.6 0)
+      (effects (font (size 1.27 1.27)) hide)
+    )
+    (property "LCSC" "" (at 154.94 101.6 0)
+      (effects (font (size 1.27 1.27)) hide)
+    )
+    (property "MyComment" "DNP" (at 149.86 105.41 0)
+      (effects (font (size 1.27 1.27)))
+    )
+    (pin "1")
+    (pin "2")
+    (instances
+      (project "uaefi"
+        (path "/ac264c30-3e9a-4be2-b97a-9949b68bd497/ced20183-e5c8-42b4-80bd-35fc70d9313a"
+          (reference "C30") (unit 1)
+        )
+      )
+    )
+  )
+  (symbol (lib_id "Power_Protection:NUP2105L") (at 119.38 101.6 0) (mirror y) (unit 1)
+    (in_bom yes) (on_board yes) (dnp no)
+    (property "Reference" "D8" (at 114.3 106.68 0)
+      (effects (font (size 1.27 1.27)) (justify left))
+    )
+    (property "Value" "NUP2105L" (at 114.3 109.22 0)
+      (effects (font (size 1.27 1.27)) (justify left))
+    )
+    (property "Footprint" "Package_TO_SOT_SMD:SOT-23" (at 113.665 102.87 0)
+      (effects (font (size 1.27 1.27)) (justify left) hide)
+    )
+    (property "Datasheet" "http://www.onsemi.com/pub_link/Collateral/NUP2105L-D.PDF" (at 116.205 98.425 0)
+      (effects (font (size 1.27 1.27)) hide)
+    )
+    (property "LCSC" "C284104" (at 119.38 101.6 0)
+      (effects (font (size 1.27 1.27)) hide)
+    )
+    (pin "3")
+    (pin "1")
+    (pin "2")
+    (instances
+      (project "uaefi"
+        (path "/ac264c30-3e9a-4be2-b97a-9949b68bd497/ced20183-e5c8-42b4-80bd-35fc70d9313a"
+          (reference "D8") (unit 1)
+        )
+      )
+    )
+  )
   (symbol (lib_id "Device:L") (at 106.68 87.63 90) (unit 1)
     (in_bom yes) (on_board yes) (dnp no)
@@
     )
   )
-  (symbol (lib_name "GND_4") (lib_id "power:GND") (at 176.53 77.47 0) (unit 1)
+  (symbol (lib_id "power:GND") (at 176.53 77.47 0) (unit 1)
     (in_bom yes) (on_board yes) (dnp no)
     (property "Reference" "#PWR0109" (at 176.53 83.82 0)
@@
     )
   )
-  (symbol (lib_name "GND_3") (lib_id "power:GND") (at 189.23 77.47 0) (unit 1)
+  (symbol (lib_id "power:GND") (at 189.23 77.47 0) (unit 1)
     (in_bom yes) (on_board yes) (dnp no)
     (property "Reference" "#PWR0110" (at 189.23 83.82 0)
@@
     )
   )
-  (symbol (lib_name "GND_5") (lib_id "power:GND") (at 139.7 107.95 0) (unit 1)
+  (symbol (lib_id "power:GND") (at 139.7 107.95 0) (unit 1)
     (in_bom yes) (on_board yes) (dnp no)
     (property "Reference" "#PWR0106" (at 139.7 114.3 0)
@@
     )
   )
-  (symbol (lib_name "GND_6") (lib_id "power:GND") (at 154.94 107.95 0) (unit 1)
+  (symbol (lib_id "power:GND") (at 154.94 107.95 0) (unit 1)
     (in_bom yes) (on_board yes) (dnp no)
     (property "Reference" "#PWR0107" (at 154.94 114.3 0)
@@
     )
   )
-  (symbol (lib_name "GND_7") (lib_id "power:GND") (at 166.37 105.41 0) (unit 1)
+  (symbol (lib_id "power:GND") (at 166.37 105.41 0) (unit 1)
     (in_bom yes) (on_board yes) (dnp no)
     (property "Reference" "#PWR0108" (at 166.37 111.76 0)

Commit message: Upd SCH
Parts:
- removed C28, C30: 10nF 50V, Capacitor_SMD:C_0402_1005Metric, symbol Device:C
- removed C29, C31: 100n, Capacitor_SMD:C_0402_1005Metric, symbol Device:C
- removed C32: 1u, Capacitor_SMD:C_0402_1005Metric, symbol Device:C
- added C? (x2): 10n, hellen-one-common:C0603, symbol hellen-one-common:Cap
- added C?: 1u, hellen-one-common:C0603, symbol hellen-one-common:Cap
- added C? (x2): 100n, hellen-one-common:C0603, symbol hellen-one-common:Cap
- D8: LCSC C284104 -> (none); MyComment (none) -> DNP
- L1, L2: LCSC C97853 -> (none); MyComment (none) -> DNP
- U4: LCSC C52028 -> (none); MyComment (none) -> DNP
Connections:
- net GND: now also C?.1, C?.1, C?.1, C?.1
- net Vcc: now also C?.2, C?.2
- net at D8.2 (K), L2.2, U4.2 (T-): now also C?.1, C?.2
- net at D8.1 (K), L1.2, U4.3 (T+): now also C?.2, C?.2

Commit message: Export
Connections:
- net at C?.1, C?.2, L2.2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: now also D8.1 (K); no longer D8.2 (K)
- net at C?.2, C?.2, L1.2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: now also D8.2 (K); no longer D8.1 (K)
Changed lines of the file:
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@@
     )
   )
-  (symbol (lib_id "Power_Protection:NUP2105L") (at 119.38 101.6 0) (mirror y) (unit 1)
+  (symbol (lib_id "Power_Protection:NUP2105L") (at 119.38 101.6 0) (unit 1)
     (in_bom yes) (on_board yes) (dnp no)
-    (property "Reference" "D8" (at 114.3 106.68 0)
+    (property "Reference" "D8" (at 120.65 105.41 0)
       (effects (font (size 1.27 1.27)) (justify left))
     )
-    (property "Value" "NUP2105L" (at 114.3 109.22 0)
+    (property "Value" "NUP2105L" (at 120.65 107.95 0)
       (effects (font (size 1.27 1.27)) (justify left))
     )
-    (property "Footprint" "Package_TO_SOT_SMD:SOT-23" (at 113.665 102.87 0)
+    (property "Footprint" "Package_TO_SOT_SMD:SOT-23" (at 125.095 102.87 0)
       (effects (font (size 1.27 1.27)) (justify left) hide)
     )
-    (property "Datasheet" "http://www.onsemi.com/pub_link/Collateral/NUP2105L-D.PDF" (at 116.205 98.425 0)
+    (property "Datasheet" "http://www.onsemi.com/pub_link/Collateral/NUP2105L-D.PDF" (at 122.555 98.425 0)
       (effects (font (size 1.27 1.27)) hide)
     )
@@
       (effects (font (size 1.27 1.27)) hide)
     )
-    (property "MyComment" "DNP" (at 112.395 111.76 0)
+    (property "MyComment" "DNP" (at 122.555 110.49 0)
       (effects (font (size 1.27 1.27)))
     )
