File: egt.kicad_sch (KiCad schematic)
At the start: 9 parts, among them U4 MAX31855KASA

Commit message: Upd PCB
Other:
- moved on the sheet: C?
Changed lines of the file:
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@@
   (junction (at 116.84 95.25) (diameter 0) (color 0 0 0 0)
   )
-  (junction (at 135.255 95.25) (diameter 0) (color 0 0 0 0)
+  (junction (at 135.89 95.25) (diameter 0) (color 0 0 0 0)
   )
   (junction (at 121.92 87.63) (diameter 0) (color 0 0 0 0)
@@
   (junction (at 189.23 68.58) (diameter 0) (color 0 0 0 0)
   )
-  (junction (at 150.495 90.17) (diameter 0) (color 0 0 0 0)
+  (junction (at 151.13 90.17) (diameter 0) (color 0 0 0 0)
   )
   (wire (pts (xy 166.37 82.55) (xy 166.37 68.58))
@@
     (stroke (width 0) (type default))
   )
-  (wire (pts (xy 142.24 87.63) (xy 150.495 87.63))
+  (wire (pts (xy 142.24 87.63) (xy 151.13 87.63))
     (stroke (width 0) (type default))
   )
@@
     (stroke (width 0) (type default))
   )
-  (wire (pts (xy 150.495 90.17) (xy 150.495 97.79))
+  (wire (pts (xy 151.13 90.17) (xy 151.13 97.79))
     (stroke (width 0) (type default))
   )
@@
     (stroke (width 0) (type default))
   )
-  (wire (pts (xy 135.255 105.41) (xy 135.255 107.95))
+  (wire (pts (xy 135.89 105.41) (xy 135.89 107.95))
     (stroke (width 0) (type default))
   )
@@
     (stroke (width 0) (type default))
   )
-  (wire (pts (xy 150.495 87.63) (xy 150.495 90.17))
+  (wire (pts (xy 151.13 87.63) (xy 151.13 90.17))
     (stroke (width 0) (type default))
   )
@@
     (stroke (width 0) (type default))
   )
-  (wire (pts (xy 116.84 95.25) (xy 135.255 95.25))
-    (stroke (width 0) (type default))
-  )
-  (wire (pts (xy 150.495 90.17) (xy 156.21 90.17))
+  (wire (pts (xy 116.84 95.25) (xy 135.89 95.25))
+    (stroke (width 0) (type default))
+  )
+  (wire (pts (xy 151.13 90.17) (xy 156.21 90.17))
     (stroke (width 0) (type default))
   )
@@
     (stroke (width 0) (type default))
   )
-  (wire (pts (xy 150.495 105.41) (xy 150.495 107.95))
+  (wire (pts (xy 151.13 105.41) (xy 151.13 107.95))
     (stroke (width 0) (type default))
   )
@@
     (stroke (width 0) (type default))
   )
-  (wire (pts (xy 135.255 95.25) (xy 142.24 95.25))
+  (wire (pts (xy 135.89 95.25) (xy 142.24 95.25))
     (stroke (width 0) (type default))
   )
@@
     (stroke (width 0) (type default))
   )
-  (wire (pts (xy 135.255 95.25) (xy 135.255 97.79))
+  (wire (pts (xy 135.89 95.25) (xy 135.89 97.79))
     (stroke (width 0) (type default))
   )
@@
     (effects (font (size 1.27 1.27)) (justify right))
   )
-  (symbol (lib_id "hellen-one-common:Cap") (at 135.255 101.6 90) (unit 1)
-    (in_bom yes) (on_board yes) (dnp no)
-    (property "Reference" "C?" (at 137.795 99.695 90)
-      (effects (font (size 1.27 1.27)) (justify right))
-    )
-    (property "Value" "10n" (at 137.795 101.6 90)
-      (effects (font (size 1.27 1.27)) (justify right))
-    )
-    (property "Footprint" "hellen-one-common:C0603" (at 139.065 104.14 0)
-      (effects (font (size 1.27 1.27)) hide)
-    )
-    (property "Datasheet" "" (at 135.255 105.41 90)
-      (effects (font (size 1.27 1.27)) hide)
-    )
-    (property "LCSC" "" (at 135.255 101.6 0)
-      (effects (font (size 1.27 1.27)) hide)
-    )
-    (property "MyComment" "DNP" (at 139.7 103.505 90)
+  (symbol (lib_id "hellen-one-common:Cap") (at 135.89 101.6 90) (unit 1)
+    (in_bom yes) (on_board yes) (dnp no)
+    (property "Reference" "C?" (at 138.43 99.695 90)
+      (effects (font (size 1.27 1.27)) (justify right))
+    )
+    (property "Value" "10n" (at 138.43 101.6 90)
+      (effects (font (size 1.27 1.27)) (justify right))
+    )
+    (property "Footprint" "hellen-one-common:C0603" (at 139.7 104.14 0)
+      (effects (font (size 1.27 1.27)) hide)
+    )
+    (property "Datasheet" "" (at 135.89 105.41 90)
+      (effects (font (size 1.27 1.27)) hide)
+    )
+    (property "LCSC" "" (at 135.89 101.6 0)
+      (effects (font (size 1.27 1.27)) hide)
+    )
+    (property "MyComment" "DNP" (at 140.335 103.505 90)
       (effects (font (size 1.27 1.27)))
     )
@@
     )
   )
-  (symbol (lib_id "hellen-one-common:Cap") (at 150.495 101.6 90) (unit 1)
-    (in_bom yes) (on_board yes) (dnp no)
-    (property "Reference" "C?" (at 153.035 99.695 90)
-      (effects (font (size 1.27 1.27)) (justify right))
-    )
-    (property "Value" "10n" (at 153.035 101.6 90)
-      (effects (font (size 1.27 1.27)) (justify right))
-    )
-    (property "Footprint" "hellen-one-common:C0603" (at 154.305 104.14 0)
-      (effects (font (size 1.27 1.27)) hide)
-    )
-    (property "Datasheet" "" (at 150.495 105.41 90)
-      (effects (font (size 1.27 1.27)) hide)
-    )
-    (property "LCSC" "" (at 150.495 101.6 0)
-      (effects (font (size 1.27 1.27)) hide)
-    )
-    (property "MyComment" "DNP" (at 154.94 103.505 90)
+  (symbol (lib_id "hellen-one-common:Cap") (at 151.13 101.6 90) (unit 1)
+    (in_bom yes) (on_board yes) (dnp no)
+    (property "Reference" "C?" (at 153.67 99.695 90)
+      (effects (font (size 1.27 1.27)) (justify right))
+    )
+    (property "Value" "10n" (at 153.67 101.6 90)
+      (effects (font (size 1.27 1.27)) (justify right))
+    )
+    (property "Footprint" "hellen-one-common:C0603" (at 154.94 104.14 0)
+      (effects (font (size 1.27 1.27)) hide)
+    )
+    (property "Datasheet" "" (at 151.13 105.41 90)
+      (effects (font (size 1.27 1.27)) hide)
+    )
+    (property "LCSC" "" (at 151.13 101.6 0)
+      (effects (font (size 1.27 1.27)) hide)
+    )
+    (property "MyComment" "DNP" (at 155.575 103.505 90)
       (effects (font (size 1.27 1.27)))
     )
@@
     )
   )
-  (symbol (lib_id "power:GND") (at 135.255 107.95 0) (unit 1)
-    (in_bom yes) (on_board yes) (dnp no)
-    (property "Reference" "#PWR0106" (at 135.255 114.3 0)
-      (effects (font (size 1.27 1.27)) hide)
-    )
-    (property "Value" "GND" (at 135.382 112.3442 0)
-      (effects (font (size 1.27 1.27)) hide)
-    )
-    (property "Footprint" "" (at 135.255 107.95 0)
-      (effects (font (size 1.27 1.27)) hide)
-    )
-    (property "Datasheet" "" (at 135.255 107.95 0)
+  (symbol (lib_id "power:GND") (at 135.89 107.95 0) (unit 1)
+    (in_bom yes) (on_board yes) (dnp no)
+    (property "Reference" "#PWR0106" (at 135.89 114.3 0)
+      (effects (font (size 1.27 1.27)) hide)
+    )
+    (property "Value" "GND" (at 136.017 112.3442 0)
+      (effects (font (size 1.27 1.27)) hide)
+    )
+    (property "Footprint" "" (at 135.89 107.95 0)
+      (effects (font (size 1.27 1.27)) hide)
+    )
+    (property "Datasheet" "" (at 135.89 107.95 0)
       (effects (font (size 1.27 1.27)) hide)
     )
@@
     )
   )
-  (symbol (lib_id "power:GND") (at 150.495 107.95 0) (unit 1)
-    (in_bom yes) (on_board yes) (dnp no)
-    (property "Reference" "#PWR0107" (at 150.495 114.3 0)
-      (effects (font (size 1.27 1.27)) hide)
-    )
-    (property "Value" "GND" (at 150.622 112.3442 0)
-      (effects (font (size 1.27 1.27)) hide)
-    )
-    (property "Footprint" "" (at 150.495 107.95 0)
-      (effects (font (size 1.27 1.27)) hide)
-    )
-    (property "Datasheet" "" (at 150.495 107.95 0)
-      (effects (font (size 1.27 1.27)) hide)
-    )
+  (symbol (lib_id "power:GND") (at 151.13 107.95 0) (unit 1)
+    (in_bom yes) (on_board yes) (dnp no)
+    (property "Reference" "#PWR0107" (at 151.13 114.3 0)
+      (effects (font (size 1.27 1.27)) hide)
+    )
+    (property "Value" "GND" (at 151.257 112.3442 0)
+      (effects (font (size 1.27 1.27)) hide)
+    )
+    (property "Footprint" "" (at 151.13 107.95 0)
+      (effects (font (size 1.27 1.27)) hide)
+    )
+    (property "Datasheet" "" (at 151.13 107.95 0)
+      (effects (font (size 1.27 1.27)) hide)
+    )

Commit message: Rev C
Parts:
- C? (x2): LCSC (none) -> C57112; MyComment DNP -> (none)
- C?: LCSC (none) -> C15849; MyComment DNP -> (none)
- C? (x2): LCSC (none) -> C14663; MyComment DNP -> (none)
- D8: LCSC (none) -> C284104; MyComment DNP -> (none)
- L1, L2: LCSC (none) -> C97853; MyComment DNP -> (none)
- U4: LCSC (none) -> C52028; MyComment DNP -> (none)
Changed lines of the file:
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@@
       (effects (font (size 1.27 1.27)) hide)
     )
-    (property "LCSC" "" (at 135.89 101.6 0)
-      (effects (font (size 1.27 1.27)) hide)
-    )
-    (property "MyComment" "DNP" (at 140.335 103.505 90)
-      (effects (font (size 1.27 1.27)))
+    (property "LCSC" "C57112" (at 135.89 101.6 0)
+      (effects (font (size 1.27 1.27)) hide)
     )
     (pin "1")
@@
       (effects (font (size 1.27 1.27)) hide)
     )
-    (property "LCSC" "" (at 166.37 92.71 0)
-      (effects (font (size 1.27 1.27)) hide)
-    )
-    (property "MyComment" "DNP" (at 176.53 84.455 0)
-      (effects (font (size 1.27 1.27)))
+    (property "LCSC" "C52028" (at 166.37 92.71 0)
+      (effects (font (size 1.27 1.27)) hide)
     )
     (pin "1")
@@
       (effects (font (size 1.27 1.27)) hide)
     )
-    (property "LCSC" "" (at 189.23 73.66 0)
-      (effects (font (size 1.27 1.27)) hide)
-    )
-    (property "MyComment" "DNP" (at 193.675 75.565 90)
-      (effects (font (size 1.27 1.27)))
+    (property "LCSC" "C15849" (at 189.23 73.66 0)
+      (effects (font (size 1.27 1.27)) hide)
     )
     (pin "1")
@@
       (effects (font (size 1.27 1.27)) hide)
     )
-    (property "LCSC" "" (at 151.13 101.6 0)
-      (effects (font (size 1.27 1.27)) hide)
-    )
-    (property "MyComment" "DNP" (at 155.575 103.505 90)
-      (effects (font (size 1.27 1.27)))
+    (property "LCSC" "C57112" (at 151.13 101.6 0)
+      (effects (font (size 1.27 1.27)) hide)
     )
     (pin "1")
@@
       (effects (font (size 1.27 1.27)) hide)
     )
-    (property "LCSC" "" (at 119.38 101.6 0)
-      (effects (font (size 1.27 1.27)) hide)
-    )
-    (property "MyComment" "DNP" (at 122.555 110.49 0)
-      (effects (font (size 1.27 1.27)))
+    (property "LCSC" "C284104" (at 119.38 101.6 0)
+      (effects (font (size 1.27 1.27)) hide)
     )
     (pin "3")
@@
       (effects (font (size 1.27 1.27)) hide)
     )
-    (property "LCSC" "" (at 176.53 73.66 0)
-      (effects (font (size 1.27 1.27)) hide)
-    )
-    (property "MyComment" "DNP" (at 180.975 75.565 90)
-      (effects (font (size 1.27 1.27)))
+    (property "LCSC" "C14663" (at 176.53 73.66 0)
+      (effects (font (size 1.27 1.27)) hide)
     )
     (pin "1")
@@
       (effects (font (size 1.27 1.27)) hide)
     )
-    (property "LCSC" "" (at 106.68 95.25 90)
-      (effects (font (size 1.27 1.27)) hide)
-    )
-    (property "MyComment" "DNP" (at 109.855 97.79 90)
-      (effects (font (size 1.27 1.27)))
+    (property "LCSC" "C97853" (at 106.68 95.25 90)
+      (effects (font (size 1.27 1.27)) hide)
     )
     (pin "1")
@@
       (effects (font (size 1.27 1.27)) hide)
     )
-    (property "LCSC" "" (at 142.24 91.44 0)
-      (effects (font (size 1.27 1.27)) hide)
-    )
-    (property "MyComment" "DNP" (at 146.685 93.345 90)
-      (effects (font (size 1.27 1.27)))
+    (property "LCSC" "C14663" (at 142.24 91.44 0)
+      (effects (font (size 1.27 1.27)) hide)
     )
     (pin "1")
@@
       (effects (font (size 1.27 1.27)) hide)
     )
-    (property "LCSC" "" (at 106.68 87.63 90)
-      (effects (font (size 1.27 1.27)) hide)
-    )
-    (property "MyComment" "DNP" (at 109.855 90.17 90)
-      (effects (font (size 1.27 1.27)))
-    )
-    (pin "1")
+    (property "LCSC" "C97853" (at 106.68 87.63 90)
+      (effects (font (size 1.27 1.27)) hide)
+    )
+    (pin "1")
