File: egt.kicad_sch (KiCad schematic)
At the start: 9 parts, among them U4 MAX31855KASA

Commit message: #66
Other:
- company: (none) -> rusEFI.com
- title: (none) -> UAEFI

Commit message: #62 #65 #66 #67 #53
Other:
- note added: "NUP2105L is optional, used for protection"
Changed lines of the file:
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@@
 	(title_block
 		(title "UAEFI")
-		(date "2024-08-14")
+		(date "2024-08-15")
 		(rev "D")
 		(company "rusEFI.com")
@@
 		)
 	)
+	(text "NUP2105L is optional, used for protection"
+		(exclude_from_sim no)
+		(at 121.412 114.808 0)
+		(effects
+			(font
+				(size 1.27 1.27)
+			)
+		)
+	)
