File: IGN6.kicad_sch (KiCad schematic)
At the start: 18 parts

Commit message: Upd SCH
Other:
- note added: "Remove R19, R21, R25, R23, R28, R29, and install Q1-Q6 for use with dumb coils"
Changed lines of the file:
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@@
     (stroke (width 0) (type default))
+  )
+  (text "Remove R19, R21, R25, R23, R28, R29, and install Q1-Q6 for use with dumb coils"
+    (at 104.14 58.42 0)
+    (effects (font (size 1.27 1.27)) (justify left bottom))
   )
   (hierarchical_label "IN5" (shape input) (at 185.42 97.79 0) (fields_autoplaced)

Commit message: Upd PCB
Parts:
- Q? (x6): value ISL9V3040D3S -> ISL9V3040D3ST
Other:
- note added: "Remove R20-R22, R26-R28, and install Q7-Q12 for use with dumb coils"
- note removed: "Remove R19, R21, R25, R23, R28, R29, and install Q1-Q6 for use with dumb coils"
Changed lines of the file:
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@@
     (stroke (width 0) (type default))
   )
-  (text "Remove R19, R21, R25, R23, R28, R29, and install Q1-Q6 for use with dumb coils"
-    (at 104.14 58.42 0)
+  (text "Remove R20-R22, R26-R28, and install Q7-Q12 for use with dumb coils"
+    (at 106.68 58.42 0)
     (effects (font (size 1.27 1.27)) (justify left bottom))
   )
@@
       (effects (font (size 1.27 1.27)) (justify left))
     )
-    (property "Value" "ISL9V3040D3S" (at 115.7986 126.873 0)
+    (property "Value" "ISL9V3040D3ST" (at 115.7986 126.873 0)
       (effects (font (size 1.27 1.27)) (justify left))
     )
@@
       (effects (font (size 1.27 1.27)) (justify left))
     )
-    (property "Value" "ISL9V3040D3S" (at 115.7986 70.993 0)
+    (property "Value" "ISL9V3040D3ST" (at 115.7986 70.993 0)
       (effects (font (size 1.27 1.27)) (justify left))
     )
@@
       (effects (font (size 1.27 1.27)) (justify left))
     )
-    (property "Value" "ISL9V3040D3S" (at 115.7986 98.933 0)
+    (property "Value" "ISL9V3040D3ST" (at 115.7986 98.933 0)
       (effects (font (size 1.27 1.27)) (justify left))
     )
@@
       (effects (font (size 1.27 1.27)) (justify left))
     )
-    (property "Value" "ISL9V3040D3S" (at 162.7886 70.993 0)
+    (property "Value" "ISL9V3040D3ST" (at 162.7886 70.993 0)
       (effects (font (size 1.27 1.27)) (justify left))
     )
@@
       (effects (font (size 1.27 1.27)) (justify left))
     )
-    (property "Value" "ISL9V3040D3S" (at 162.7886 126.873 0)
+    (property "Value" "ISL9V3040D3ST" (at 162.7886 126.873 0)
       (effects (font (size 1.27 1.27)) (justify left))
     )
@@
       (effects (font (size 1.27 1.27)) (justify left))
     )
-    (property "Value" "ISL9V3040D3S" (at 162.7886 98.933 0)
-      (effects (font (size 1.27 1.27)) (justify left))
-    )
+    (property "Value" "ISL9V3040D3ST" (at 162.7886 98.933 0)
+      (effects (font (size 1.27 1.27)) (justify left))
+    )

Commit message: Upd PCB
Parts:
- added F10, F5, F6, F7, F8, F9: 50mA, Fuse:Fuse_0603_1608Metric, symbol Device:Polyfuse
Connections:
- net IN1: now also F6.2; no longer R14.1, R7.2
- net IN2: now also F5.2; no longer R14.1, R7.2
- net IN3: now also F7.2; no longer R14.1, R7.2
- net IN4: now also F8.2; no longer R14.1, R7.2
- net IN5: now also F9.2; no longer R14.1, R7.2
- net IN6: now also F10.2; no longer R14.1, R7.2
- new net: F9.1, R14.1, R7.2
- new net: F10.1, R14.1, R7.2
- new net: F6.1, R14.1, R7.2
- new net: F8.1, R14.1, R7.2
- new net: F5.1, R14.1, R7.2
- new net: F7.1, R14.1, R7.2

Commit message: #66
Other:
- company: rusefi.com -> rusEFI.com
- title: UAEFI Ignition -> UAEFI
