File: DC_MOTOR_0.1.kicad_sch (KiCad schematic)
At the start: 15 parts

Commit message: Upd PCB
Parts:
- added P3 (x2): Pad, hellen-one-common:PAD-TH, symbol hellen-one-common:Pad
Connections:
- net DIR: now also P3.1 (Pin_1)
- net PWM: now also P3.1 (Pin_1)
Changed lines of the file:
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@@
   (junction (at 135.89 80.01) (diameter 0) (color 0 0 0 0)
+  )
+  (junction (at 215.9 106.68) (diameter 0) (color 0 0 0 0)
+  )
+  (junction (at 215.9 104.14) (diameter 0) (color 0 0 0 0)
   )
   (junction (at 203.2 116.84) (diameter 0) (color 0 0 0 0)
@@
     (stroke (width 0) (type default))
   )
-  (wire (pts (xy 203.2 106.68) (xy 227.33 106.68))
+  (wire (pts (xy 203.2 106.68) (xy 215.9 106.68))
     (stroke (width 0) (type default))
   )
@@
     (stroke (width 0) (type default))
   )
+  (wire (pts (xy 215.9 104.14) (xy 215.9 105.41))
+    (stroke (width 0) (type default))
+  )
   (wire (pts (xy 203.2 114.3) (xy 203.2 116.84))
     (stroke (width 0) (type default))
@@
     (stroke (width 0) (type default))
   )
-  (wire (pts (xy 203.2 104.14) (xy 227.33 104.14))
+  (wire (pts (xy 203.2 104.14) (xy 215.9 104.14))
     (stroke (width 0) (type default))
   )
   (wire (pts (xy 91.44 80.01) (xy 100.33 80.01))
+    (stroke (width 0) (type default))
+  )
+  (wire (pts (xy 215.9 104.14) (xy 227.33 104.14))
+    (stroke (width 0) (type default))
+  )
+  (wire (pts (xy 215.9 106.68) (xy 227.33 106.68))
     (stroke (width 0) (type default))
   )
@@
   )
   (wire (pts (xy 182.88 80.01) (xy 182.88 96.52))
+    (stroke (width 0) (type default))
+  )
+  (wire (pts (xy 215.9 106.68) (xy 215.9 107.95))
     (stroke (width 0) (type default))
   )
@@
     )
   )
+  (symbol (lib_id "hellen-one-common:Pad") (at 220.98 107.95 0) (unit 1)
+    (in_bom yes) (on_board yes) (dnp no)
+    (property "Reference" "P3" (at 222.25 107.95 0)
+      (effects (font (size 1.27 1.27)) (justify left))
+    )
+    (property "Value" "Pad" (at 220.98 110.49 0)
+      (effects (font (size 1.27 1.27)) hide)
+    )
+    (property "Footprint" "hellen-one-common:PAD-TH" (at 220.98 111.76 0)
+      (effects (font (size 1.27 1.27)) hide)
+    )
+    (property "Datasheet" "~" (at 220.98 107.95 0)
+      (effects (font (size 1.27 1.27)) hide)
+    )
+    (pin "1")
+    (instances
+      (project "uaefi"
+        (path "/ac264c30-3e9a-4be2-b97a-9949b68bd497"
+          (reference "P3") (unit 1)
+        )
+        (path "/ac264c30-3e9a-4be2-b97a-9949b68bd497/0c617583-4e3e-4059-8607-2ed650d520f4"
+          (reference "P15") (unit 1)
+        )
+        (path "/ac264c30-3e9a-4be2-b97a-9949b68bd497/b2716558-3a44-4e63-a5d7-5409c167071f"
+          (reference "P16") (unit 1)
+        )
+      )
+    )
+  )
   (symbol (lib_id "hellen-one-common:Cap") (at 127 83.82 90) (unit 1)
     (in_bom yes) (on_board yes) (dnp no)
@@
         )
       )
+    )
+  )
+  (symbol (lib_id "hellen-one-common:Pad") (at 220.98 105.41 0) (unit 1)
+    (in_bom yes) (on_board yes) (dnp no)
+    (property "Reference" "P3" (at 222.25 105.41 0)
+      (effects (font (size 1.27 1.27)) (justify left))
+    )
+    (property "Value" "Pad" (at 220.98 107.95 0)
+      (effects (font (size 1.27 1.27)) hide)
+    )
+    (property "Footprint" "hellen-one-common:PAD-TH" (at 220.98 109.22 0)
+      (effects (font (size 1.27 1.27)) hide)
+    )
+    (property "Datasheet" "~" (at 220.98 105.41 0)
+      (effects (font (size 1.27 1.27)) hide)
+    )
+    (pin "1")
+    (instances
+      (project "uaefi"
+        (path "/ac264c30-3e9a-4be2-b97a-9949b68bd497"
+          (reference "P3") (unit 1)
+        )
+        (path "/ac264c30-3e9a-4be2-b97a-9949b68bd497/0c617583-4e3e-4059-8607-2ed650d520f4"
+          (reference "P17") (unit 1)
+        )
+        (path "/ac264c30-3e9a-4be2-b97a-9949b68bd497/b2716558-3a44-4e63-a5d7-5409c167071f"
+          (reference "P18") (unit 1)
+        )
+      )

Commit message: Upd PCB
Parts:
- renumbered P3 to P15, P3 to P17
Changed lines of the file:
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@@
   (symbol (lib_id "hellen-one-common:Pad") (at 220.98 107.95 0) (unit 1)
     (in_bom yes) (on_board yes) (dnp no)
-    (property "Reference" "P3" (at 222.25 107.95 0)
+    (property "Reference" "P15" (at 222.25 107.95 0)
       (effects (font (size 1.27 1.27)) (justify left))
     )
@@
     (instances
       (project "uaefi"
-        (path "/ac264c30-3e9a-4be2-b97a-9949b68bd497"
-          (reference "P3") (unit 1)
-        )
         (path "/ac264c30-3e9a-4be2-b97a-9949b68bd497/0c617583-4e3e-4059-8607-2ed650d520f4"
           (reference "P15") (unit 1)
@@
   (symbol (lib_id "hellen-one-common:Pad") (at 220.98 105.41 0) (unit 1)
     (in_bom yes) (on_board yes) (dnp no)
-    (property "Reference" "P3" (at 222.25 105.41 0)
+    (property "Reference" "P17" (at 222.25 105.41 0)
       (effects (font (size 1.27 1.27)) (justify left))
     )
@@
     (instances
       (project "uaefi"
-        (path "/ac264c30-3e9a-4be2-b97a-9949b68bd497"
-          (reference "P3") (unit 1)
-        )
         (path "/ac264c30-3e9a-4be2-b97a-9949b68bd497/0c617583-4e3e-4059-8607-2ed650d520f4"
           (reference "P17") (unit 1)

Commit message: #66
Other:
- company: rusefi.com -> rusEFI.com
- title: UAEFI DC motor driver -> UAEFI

Commit message: Rev E
Other:
- moved on the sheet: R?
Changed lines of the file:
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@@
 	(title_block
 		(title "UAEFI")
-		(date "2024-08-15")
-		(rev "D")
+		(date "2025-04-30")
+		(rev "E")
 		(company "rusEFI.com")
 	)
@@
 	)
 	(junction
-		(at 219.71 91.44)
+		(at 219.71 88.9)
 		(diameter 0)
 		(color 0 0 0 0)
@@
 	)
 	(junction
+		(at 203.2 114.3)
+		(diameter 0)
+		(color 0 0 0 0)
+	)
+	(junction
 		(at 175.26 106.68)
 		(diameter 0)
@@
 	)
 	(junction
-		(at 203.2 114.3)
-		(diameter 0)
-		(color 0 0 0 0)
-	)
-	(junction
 		(at 162.56 80.01)
 		(diameter 0)
@@
 	(wire
 		(pts
-			(xy 203.2 96.52) (xy 213.36 96.52)
-		)
-		(stroke
-			(width 0)
-			(type default)
-		)
-	)
-	(wire
-		(pts
-			(xy 203.2 111.76) (xy 203.2 114.3)
-		)
-		(stroke
-			(width 0)
-			(type default)
-		)
-	)
-	(wire
-		(pts
 			(xy 203.2 106.68) (xy 215.9 106.68)
 		)
@@
 	(wire
 		(pts
-			(xy 203.2 114.3) (xy 203.2 116.84)
+			(xy 203.2 114.3) (xy 203.2 111.76)
 		)
 		(stroke
@@
 	(wire
 		(pts
-			(xy 219.71 91.44) (xy 227.33 91.44)
+			(xy 219.71 88.9) (xy 227.33 88.9)
 		)
 		(stroke
@@
 	(wire
 		(pts
-			(xy 213.36 96.52) (xy 213.36 91.44)
+			(xy 203.2 96.52) (xy 203.2 88.9)
 		)
 		(stroke
@@
 	(wire
 		(pts
+			(xy 219.71 99.06) (xy 219.71 101.6)
+		)
+		(stroke
+			(width 0)
+			(type default)
+		)
+	)
+	(wire
+		(pts
 			(xy 82.55 80.01) (xy 91.44 80.01)
 		)
@@
 	(wire
 		(pts
+			(xy 203.2 116.84) (xy 203.2 114.3)
+		)
+		(stroke
+			(width 0)
+			(type default)
+		)
+	)
+	(wire
+		(pts
 			(xy 135.89 80.01) (xy 144.78 80.01)
 		)
@@
 	(wire
 		(pts
-			(xy 213.36 91.44) (xy 219.71 91.44)
+			(xy 203.2 88.9) (xy 219.71 88.9)
 		)
 		(stroke
@@
 	(hierarchical_label "3V3"
 		(shape passive)
-		(at 227.33 91.44 0)
+		(at 227.33 88.9 0)
 		(fields_autoplaced yes)
 		(effects
@@
 			)
 		)
-		(property "Description" ""
+		(property "Description" "Power symbol creates a global label with name \"GND\" , ground"
 			(at 118.11 87.63 0)
 			(effects
@@
 	)
 	(symbol
+		(lib_id "power:GND")
+		(at 203.2 116.84 90)
+		(mirror x)
+		(unit 1)
+		(exclude_from_sim no)
+		(in_bom yes)
+		(on_board yes)
+		(dnp no)
+		(fields_autoplaced yes)
+		(property "Reference" "#PWR066"
+			(at 209.55 116.84 0)
+			(effects
+				(font
+					(size 1.27 1.27)
+				)
+				(hide yes)
+			)
+		)
+		(property "Value" "GND"
+			(at 207.01 116.8399 90)
+			(effects
+				(font
+					(size 1.27 1.27)
+				)
+				(justify right)
+			)
+		)
+		(property "Footprint" ""
+			(at 203.2 116.84 0)
+			(effects
+				(font
+					(size 1.27 1.27)
+				)
+				(hide yes)
+			)
+		)
+		(property "Datasheet" ""
+			(at 203.2 116.84 0)
+			(effects
+				(font
+					(size 1.27 1.27)
+				)
+				(hide yes)
+			)
+		)
+		(property "Description" "Power symbol creates a global label with name \"GND\" , ground"
+			(at 203.2 116.84 0)
+			(effects
+				(font
+					(size 1.27 1.27)
+				)
+				(hide yes)
+			)
+		)
+		(pin "1"
+		)
+		(instances
+			(project "uaefi"
+				(path "/ac264c30-3e9a-4be2-b97a-9949b68bd497/0c617583-4e3e-4059-8607-2ed650d520f4"
+					(reference "#PWR066")
+					(unit 1)
+				)
+				(path "/ac264c30-3e9a-4be2-b97a-9949b68bd497/b2716558-3a44-4e63-a5d7-5409c167071f"
+					(reference "#PWR089")
+					(unit 1)
+				)
+			)
+		)
+	)
+	(symbol
 		(lib_id "hellen-one-common:Cap")
 		(at 118.11 83.82 90)
@@
 			)
 		)
-		(property "Description" ""
+		(property "Description" "Power symbol creates a global label with name \"GND\" , ground"
 			(at 144.78 87.63 0)
 			(effects
@@
 			)
 		)
-		(property "Description" ""
+		(property "Description" "Power symbol creates a global label with name \"GND\" , ground"
 			(at 91.44 87.63 0)
 			(effects
@@
 	(symbol
 		(lib_id "hellen-one-common:Res")
-		(at 219.71 101.6 90)
+		(at 219.71 99.06 90)
 		(unit 1)
 		(exclude_from_sim no)
@@
 		(dnp no)
 		(property "Reference" "R?"
-			(at 222.25 96.52 0)
+			(at 222.25 93.98 0)
 			(effects
 				(font
@@
 		)
 		(property "Value" "4.7k"
-			(at 219.71 96.52 0)
+			(at 219.71 93.98 0)
 			(effects
 				(font
@@
 		)
 		(property "Footprint" "hellen-one-common:R0603"
-			(at 223.52 97.79 0)
+			(at 223.52 95.25 0)
 			(effects
 				(font
@@
 		)
 		(property "Datasheet" ""
-			(at 219.71 101.6 0)
+			(at 219.71 99.06 0)
 			(effects
 				(font
@@
 		)
 		(property "Description" ""
-			(at 219.71 101.6 0)
+			(at 219.71 99.06 0)
 			(effects
 				(font
@@
 		)
 		(property "LCSC" "C23162"
-			(at 219.71 101.6 0)
+			(at 219.71 99.06 0)
 			(effects
 				(font
@@
 			)
 		)
-		(property "Description" ""
+		(property "Description" "Power symbol creates a global label with name \"GND\" , ground"
 			(at 127 87.63 0)
 			(effects
@@
 	(symbol
 		(lib_id "power:GND")
-		(at 203.2 116.84 90)
-		(mirror x)
-		(unit 1)
-		(exclude_from_sim no)
-		(in_bom yes)
-		(on_board yes)
-		(dnp no)
-		(property "Reference" "#PWR?"
-			(at 209.55 116.84 0)
-			(effects
-				(font
-					(size 1.27 1.27)
-				)
-				(hide yes)
-			)
-		)
-		(property "Value" "GND"
-			(at 207.01 116.84 90)
-			(effects
-				(font
-					(size 1.27 1.27)
-				)
-				(justify right)
-			)
-		)
-		(property "Footprint" ""
-			(at 203.2 116.84 0)
-			(effects
-				(font
-					(size 1.27 1.27)
-				)
-				(hide yes)
-			)
-		)
-		(property "Datasheet" ""
-			(at 203.2 116.84 0)
-			(effects
-				(font
-					(size 1.27 1.27)
-				)
-				(hide yes)
-			)
-		)
-		(property "Description" ""
-			(at 203.2 116.84 0)
-			(effects
-				(font
-					(size 1.27 1.27)
-				)
-				(hide yes)
-			)
-		)
-		(pin "1"
-		)
-		(instances
-			(project "hellen-112-17"
-				(path "/63d2dd9f-d5ff-4811-a88d-0ba932475460"
-					(reference "#PWR?")
-					(unit 1)
-				)
-				(path "/63d2dd9f-d5ff-4811-a88d-0ba932475460/61fdb358-02a6-4f6d-a5c3-cab9f97fc6da"
-					(reference "#PWR?")
-					(unit 1)
-				)
-			)
-			(project "uaefi"
-				(path "/ac264c30-3e9a-4be2-b97a-9949b68bd497/0c617583-4e3e-4059-8607-2ed650d520f4"
-					(reference "#PWR066")
-					(unit 1)
-				)
-				(path "/ac264c30-3e9a-4be2-b97a-9949b68bd497/b2716558-3a44-4e63-a5d7-5409c167071f"
-					(reference "#PWR089")
-					(unit 1)
-				)
-			)
-		)
-	)
-	(symbol
-		(lib_id "power:GND")
 		(at 100.33 87.63 0)
 		(unit 1)
@@
 			)
 		)
-		(property "Description" ""
+		(property "Description" "Power symbol creates a global label with name \"GND\" , ground"
 			(at 100.33 87.63 0)
 			(effects
@@
 			)
 		)
-		(property "Description" ""
+		(property "Description" "Power symbol creates a global label with name \"GND\" , ground"
 			(at 153.67 87.63 0)
 			(effects
@@
 			)
 		)
-		(property "Description" ""
+		(property "Description" "Power symbol creates a global label with name \"GND\" , ground"
 			(at 109.22 87.63 0)
 			(effects
@@
 			)
 		)
-		(property "Description" ""
+		(property "Description" "Power symbol creates a global label with name \"GND\" , ground"
 			(at 73.66 87.63 0)
 			(effects
@@
 			)
 		)
-		(property "Description" ""
+		(property "Description" "Power symbol creates a global label with name \"GND\" , ground"
 			(at 175.26 115.57 0)
 			(effects
@@
 			)
 		)
-		(property "Description" ""
+		(property "Description" "Power symbol creates a global label with name \"GND\" , ground"
 			(at 175.26 88.9 0)
 			(effects
@@
 			)
 		)
-		(property "Description" ""
+		(property "Description" "Power symbol creates a global label with name \"GND\" , ground"
 			(at 182.88 121.92 0)
 			(effects
@@
 			)
 		)
-		(property "Description" ""
+		(property "Description" "Power symbol creates a global label with name \"GND\" , ground"
 			(at 162.56 87.63 0)
 			(effects
@@
 			)
 		)
-		(property "Description" ""
+		(property "Description" "Power symbol creates a global label with name \"GND\" , ground"
 			(at 82.55 87.63 0)
 			(effects
@@
 			)
 		)
-		(property "Description" ""
+		(property "Description" "Power symbol creates a global label with name \"GND\" , ground"
 			(at 135.89 87.63 0)
 			(effects
