File: MAP.kicad_sch (KiCad schematic)
At the start: 2 parts, among them U3 MPXH6400A

Commit message: Upd SCH
Parts:
- removed U3: MPXH6400A, hellen-one-common:MPXH6400A-SSOP8, symbol MPX-4_MAP:MPX4_MAP
- added U3: MPX4/MPXH6400_MAP, kicad6-libraries:MPX-4_MAP, symbol MPX-4_MAP:MPX4/MPXH6400_MAP
Connections:
- net +5VA: now also U3.3 (VCC)
- net GND: now also U3.2 (GND)
- net OUT: now also U3.1 (VOUT)
- no-connect marks 5 -> 3
Changed lines of the file:
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@@
   (junction (at 165.1 88.9) (diameter 0) (color 0 0 0 0)
   )
-  (no_connect (at 129.54 83.82))
-  (no_connect (at 129.54 91.44))
-  (no_connect (at 129.54 88.9))
-  (no_connect (at 129.54 86.36))
   (no_connect (at 154.94 91.44))
+  (no_connect (at 154.94 96.52))
+  (no_connect (at 154.94 93.98))
   (wire (pts (xy 165.1 88.9) (xy 154.94 88.9))
     (stroke (width 0) (type solid))
@@
         (path "/ac264c30-3e9a-4be2-b97a-9949b68bd497/7f618b1f-fe11-49db-a473-d0b521b1fa4f"
           (reference "#PWR041") (unit 1)
-        )
-      )
-    )
-  )
-  (symbol (lib_id "MPX-4_MAP:MPX4_MAP") (at 146.05 85.09 180) (unit 1)
-    (in_bom yes) (on_board yes) (dnp no)
-    (property "Reference" "U3" (at 142.24 78.74 0)
-      (effects (font (size 1.524 1.524)) (justify left))
-    )
-    (property "Value" "MPXH6400A" (at 149.86 81.28 0)
-      (effects (font (size 1.524 1.524)) (justify left))
-    )
-    (property "Footprint" "hellen-one-common:MPXH6400A-SSOP8" (at 146.05 85.09 0)
-      (effects (font (size 1.27 1.27)) hide)
-    )
-    (property "Datasheet" "" (at 146.05 85.09 0)
-      (effects (font (size 1.524 1.524)) hide)
-    )
-    (property "LCSC" "C511770" (at 146.05 85.09 0)
-      (effects (font (size 1.27 1.27)) hide)
-    )
-    (pin "1")
-    (pin "2")
-    (pin "3")
-    (pin "4")
-    (pin "5")
-    (pin "6")
-    (pin "7")
-    (pin "8")
-    (instances
-      (project "alphax_4ch"
-        (path "/63d2dd9f-d5ff-4811-a88d-0ba932475460"
-          (reference "U3") (unit 1)
-        )
-        (path "/63d2dd9f-d5ff-4811-a88d-0ba932475460/aafb5e2e-7f5c-429b-85e5-76b90069790c"
-          (reference "U3") (unit 1)
-        )
-      )
-      (project "uaefi"
-        (path "/ac264c30-3e9a-4be2-b97a-9949b68bd497/7f618b1f-fe11-49db-a473-d0b521b1fa4f"
-          (reference "U3") (unit 1)
         )
       )
@@
         )
       )
+    )
+  )
+  (symbol (lib_id "MPX-4_MAP:MPX4{slash}MPXH6400_MAP") (at 146.05 90.17 0) (mirror y) (unit 1)
+    (in_bom yes) (on_board yes) (dnp no) (fields_autoplaced)
+    (property "Reference" "U3" (at 142.24 77.47 0)
+      (effects (font (size 1.524 1.524)))
+    )
+    (property "Value" "MPX4/MPXH6400_MAP" (at 142.24 80.01 0)
+      (effects (font (size 1.524 1.524)))
+    )
+    (property "Footprint" "kicad6-libraries:MPX-4_MAP" (at 146.05 90.17 0)
+      (effects (font (size 1.27 1.27)) hide)
+    )
+    (property "Datasheet" "" (at 146.05 90.17 0)
+      (effects (font (size 1.524 1.524)) hide)
+    )
+    (pin "1")
+    (pin "2")
+    (pin "3")
+    (pin "4")
+    (pin "5")
+    (pin "6")
+    (instances
+      (project "uaefi"
+        (path "/ac264c30-3e9a-4be2-b97a-9949b68bd497/7f618b1f-fe11-49db-a473-d0b521b1fa4f"
+          (reference "U3") (unit 1)
+        )
+      )

Commit message: Upd PCB
Parts:
- U3: symbol MPX-4_MAP:MPX4/MPXH6400_MAP -> MPX-4_MAP:MPX4/MPXH6400_MAP
Changed lines of the file:
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@@
     )
   )
-  (symbol (lib_id "MPX-4_MAP:MPX4{slash}MPXH6400_MAP") (at 146.05 90.17 0) (mirror y) (unit 1)
+  (symbol (lib_id "MPX-4_MAP:MPX4/MPXH6400_MAP") (at 146.05 90.17 0) (mirror y) (unit 1)
     (in_bom yes) (on_board yes) (dnp no) (fields_autoplaced)
     (property "Reference" "U3" (at 142.24 77.47 0)

Commit message: #66
Other:
- company: (none) -> rusEFI.com
- title: (none) -> UAEFI
